Commit message: now HyperDog can handshake using gamepad btn A and right joystic

File: hyperdog_gazebo_sim/description/hyperdog_urdf_links.xacro (robot description, xacro)
@@ -33,5 +33,7 @@
                 <xacro:rightHip_mesh></xacro:rightHip_mesh>
             </geometry>
-            <material name="blue" />
+            <material name="red">
+                <color rgba="0.8 0.2 0.2 1"/>
+            </material>
         </visual>
         <collision>
@@ -50,5 +52,7 @@
                 <xacro:rightUleg_mesh></xacro:rightUleg_mesh>
             </geometry>
-            <material name="orange" />
+            <material name="orange">
+                <color rgba="0.8 0.5 0.8 1"/>
+            </material>
         </visual>
         <collision>
@@ -67,5 +71,7 @@
                 <xacro:lleg_mesh></xacro:lleg_mesh>
             </geometry>
-            <material name="red" />
+            <material name="yellow">
+                <color rgba="0.8 1.0 0.1 1"/>
+            </material>
         </visual>
         <collision>
@@ -82,10 +88,12 @@
     <!-- *********** FL_hip ********** -->
     <link name="FL_hip_link">
-        <visual>
-            <origin xyz="0 0 0" rpy="0 0 0"/>
-            <geometry>
-                <xacro:leftHip_mesh></xacro:leftHip_mesh>
-            </geometry>
-            <material name="blue" />
+        <visual>curve
+            <origin xyz="0 0 0" rpy="0 0 0"/>
+            <geometry>
+                <xacro:leftHip_mesh></xacro:leftHip_mesh>
+            </geometry>
+            <material name="red">
+                <color rgba="0.8 0.2 0.2 1"/>
+            </material>
         </visual>
         <collision>
@@ -104,5 +112,7 @@
                 <xacro:leftUleg_mesh></xacro:leftUleg_mesh>
             </geometry>
-            <material name="orange" />
+            <material name="orange">
+                <color rgba="0.8 0.5 0.8 1"/>
+            </material>
         </visual>
         <collision>
@@ -121,5 +131,7 @@
                 <xacro:lleg_mesh></xacro:lleg_mesh>
             </geometry>
-            <material name="red" />
+            <material name="yellow">
+                <color rgba="0.8 1.0 0.1 1"/>
+            </material>
         </visual>
         <collision>
@@ -141,5 +153,7 @@
                 <xacro:rightHip_mesh></xacro:rightHip_mesh>
             </geometry>
-            <material name="blue" />
+            <material name="red">
+                <color rgba="0.8 0.2 0.2 1"/>
+            </material>
         </visual>
         <collision>
@@ -158,5 +172,7 @@
                 <xacro:rightUleg_mesh></xacro:rightUleg_mesh>
             </geometry>
-            <material name="orange" />
+            <material name="orange">
+                <color rgba="0.8 0.5 0.8 1"/>
+            </material>
         </visual>
         <collision>
@@ -175,5 +191,7 @@
                 <xacro:lleg_mesh></xacro:lleg_mesh>
             </geometry>
-            <material name="red" />
+            <material name="yellow">
+                <color rgba="0.8 1.0 0.1 1"/>
+            </material>
         </visual>
         <collision>
@@ -195,5 +213,7 @@
                 <xacro:leftHip_mesh></xacro:leftHip_mesh>
             </geometry>
-            <material name="blue" />
+            <material name="red">
+                <color rgba="0.8 0.2 0.2 1"/>
+            </material>
         </visual>
         <collision>
@@ -215,5 +235,7 @@
                 <xacro:leftUleg_mesh></xacro:leftUleg_mesh>
             </geometry>
-            <material name="orange" />
+            <material name="orange">
+                <color rgba="0.8 0.5 0.8 1"/>
+            </material>
         </visual>
         <collision>
@@ -235,5 +257,7 @@
                 <xacro:lleg_mesh></xacro:lleg_mesh>
             </geometry>
-            <material name="red" />
+            <material name="yellow">
+                <color rgba="0.8 1.0 0.1 1"/>
+            </material>
         </visual>
         <collision>
