Commit message: gazebo simulation model issues fixed 1.dynamic friction reduced 2.joint torque added 3.robot feet collison points and friction added 4. gazebo test world file configuration changed

File: hyperdog_gazebo_sim/description/gazebo_ros2_control_plugin.xacro (robot description, xacro)
@@ -151,4 +151,43 @@
           <parameters>$(find hyperdog_gazebo_sim)/config/hyperdog_joint_controller.yaml</parameters>
         </plugin>
+         <plugin name="p3d_base_controller" filename="libgazebo_ros_p3d.so">
+         <ros>
+            <namespace>hyperdog</namespace>
+            <remapping>odom:=odom</remapping>
+            </ros>
+         <frame_name>map</frame_name>
+            <body_name>base_link</body_name>
+            <update_rate>200.0</update_rate>
+            <gaussian_noise>0.0</gaussian_noise>
+        <alwaysOn>true</alwaysOn>
+        <xyzOffsets>0 0 0</xyzOffsets>
+        <rpyOffsets>0 0 0</rpyOffsets>
+        </plugin>
     </gazebo>
+    <!--plugin name="imu_plugin" filename="libgazebo_ros_imu.so">
+      <alwaysOn>true</alwaysOn>
+      <body_name>imu_link</body_name>
+      <frame_name>imu_link</frame_name>
+      <topic_name>imu</topic_name>
+      <serviceName>imu_service</serviceName>
+      <gaussianNoise>0.0</gaussianNoise>
+      <updateRate>0</updateRate>
+      <imu>
+        <noise>
+          <type>gaussian</type>
+          <rate>
+            <mean>0.0</mean>
+            <stddev>2e-4</stddev>
+            <bias_mean>0.0000075</bias_mean>
+            <bias_stddev>0.0000008</bias_stddev>
+          </rate>
+          <accel>
+            <mean>0.0</mean>
+            <stddev>1.7e-2</stddev>
+            <bias_mean>0.1</bias_mean>
+            <bias_stddev>0.001</bias_stddev>
+          </accel>
+        </noise>
+      </imu>
+    </plugin-->
 </robot>

File: hyperdog_gazebo_sim/description/hyperdog_gazebo.xacro (robot description, xacro)
@@ -12,48 +12,109 @@
     <xacro:include filename="physics.xacro" />
     <gazebo reference="base_link">
+    <selfCollide>false</selfCollide>
+      <mu1 value="0.05" />
+      <mu2 value="0.05" />
         <material>Gazebo/DarkGrey  </material>
     </gazebo>
     <gazebo reference="FR_hip_link">
+    <mu1>0.2</mu1>
+    <mu2>0.2</mu2>
         <material>Gazebo/PioneerBody</material>
     </gazebo>
     <gazebo reference="FL_hip_link">
+    <mu1>0.2</mu1>
+    <mu2>0.2</mu2>
         <material>Gazebo/PioneerBody</material>
     </gazebo>
     <gazebo reference="BR_hip_link">
+    <mu1>0.2</mu1>
+    <mu2>0.2</mu2>
         <material>Gazebo/PioneerBody</material>
     </gazebo>
     <gazebo reference="BL_hip_link">
+    <mu1>0.2</mu1>
+    <mu2>0.2</mu2>
         <material>Gazebo/PioneerBody</material>
     </gazebo>
     <gazebo reference="FR_uleg_link">
+    <mu1>0.2</mu1>
+    <mu2>0.2</mu2>
         <material>Gazebo/Orange     </material>
     </gazebo>
     <gazebo reference="FL_uleg_link">
+    <mu1>0.2</mu1>
+    <mu2>0.2</mu2>
         <material>Gazebo/Orange   </material>
     </gazebo>
     <gazebo reference="BR_uleg_link">
+    <mu1>0.2</mu1>
+    <mu2>0.2</mu2>
         <material>Gazebo/Orange   </material>
     </gazebo>
     <gazebo reference="BL_uleg_link">
+    <mu1>0.2</mu1>
+    <mu2>0.2</mu2>
         <material>Gazebo/Orange </material>
     </gazebo>
     <gazebo reference="FR_lleg_link">
+    <mu1>0.2</mu1>
+    <mu2>0.2</mu2>
         <material>Gazebo/DarkYellow</material>
         <xacro:foot_surface></xacro:foot_surface>
     </gazebo>
     <gazebo reference="FL_lleg_link">
+    <mu1>0.2</mu1>
+    <mu2>0.2</mu2>
         <material>Gazebo/DarkYellow</material>
         <xacro:foot_surface></xacro:foot_surface>
     </gazebo>
     <gazebo reference="BR_lleg_link">
+    <mu1>0.2</mu1>
+    <mu2>0.2</mu2>
         <material>Gazebo/DarkYellow</material>
         <xacro:foot_surface></xacro:foot_surface>
     </gazebo>
     <gazebo reference="BL_lleg_link">
+    <mu1>0.2</mu1>
+    <mu2>0.2</mu2>
         <material>Gazebo/DarkYellow</material>
         <xacro:foot_surface></xacro:foot_surface>
     </gazebo>
-    <gazebo reference="FR_lleg_joint">
+    <!--gazebo reference="FR_lleg_joint">
+    <mu1>0.1</mu1>
+    <mu2>0.1</mu2>
+    <kp>500000.0</kp>
+    <kd>10.0</kd>
+    <minDepth>0.001</minDepth>
+    <fdir1>1 0 0</fdir1>
         <implicitSpringDamper>2</implicitSpringDamper>
-    </gazebo>
+    </gazebo-->
+    <!--gazebo reference="imu_link">
+    <plugin name="imu_plugin" filename="libgazebo_ros_imu.so">
+      <alwaysOn>true</alwaysOn>
+      <bodyName>imu_link</bodyName>
+      <frameName>imu_link</frameName>
+      <topicName>imu</topicName>
+      <serviceName>imu_service</serviceName>
+      <gaussianNoise>0.0</gaussianNoise>
+      <updateRate>0</updateRate>
+      <imu>
+        <noise>
+          <type>gaussian</type>
+          <rate>
+            <mean>0.0</mean>
+            <stddev>2e-4</stddev>
+            <bias_mean>0.0000075</bias_mean>
+            <bias_stddev>0.0000008</bias_stddev>
+          </rate>
+          <accel>
+            <mean>0.0</mean>
+            <stddev>1.7e-2</stddev>
+            <bias_mean>0.1</bias_mean>
+            <bias_stddev>0.001</bias_stddev>
+          </accel>
+        </noise>
+      </imu>
+    </plugin>
+  </gazebo-->
 </robot>

File: hyperdog_gazebo_sim/description/hyperdog_urdf_joints.xacro (robot description, xacro)
@@ -12,4 +12,9 @@
         <child link="inertial_link"/>
     </joint>
+	<joint name="imu_joint" type="fixed">
+	  <origin xyz="0 0 0" rpy="0 0 0"/>
+	  <parent link="base_link"/>
+	  <child link="imu_link"/>
+	</joint>
     <!-- *********  FR_hip  ********* -->
     <joint name="FR_hip_joint" type="revolute">
@@ -19,5 +24,5 @@
         <child link="FR_hip_link"/>
         <limit lower="-1.57" upper="1.57" velocity="1" effort="7"/>
-        <dynamics friction="10.0"/>
+        <dynamics friction="1.0"/>
     </joint>
     <!-- *********  FR_uleg  ********* -->
@@ -28,5 +33,5 @@
         <child link="FR_uleg_link"/>
         <limit lower="-1.2217" upper="3.14" velocity="1" effort="7"/>
-        <dynamics friction="10.0"/>
+        <dynamics friction="1.0"/>
     </joint>
     <!-- *********  FR_lleg  ********* -->
@@ -46,5 +51,5 @@
         <child link="FL_hip_link"/>
         <limit lower="-1.57" upper="1.57" velocity="1" effort="7"/>
-        <dynamics friction="10.0"/>
+        <dynamics friction="1.0"/>
     </joint>
     <!-- *********  FL_uleg  ********* -->
@@ -55,5 +60,5 @@
         <child link="FL_uleg_link"/>
         <limit lower="-1.2217" upper="3.14" velocity="1" effort="7"/>
-        <dynamics friction="10.0"/>
+        <dynamics friction="1.0"/>
     </joint>
     <!-- *********  FL_lleg  ********* -->
@@ -73,5 +78,5 @@
         <child link="BR_hip_link"/>
         <limit lower="-1.57" upper="1.57" velocity="1" effort="7"/>
-        <dynamics friction="10.0"/>
+        <dynamics friction="1.0"/>
     </joint>
     <!-- *********  BR_uleg  ********* -->
@@ -82,5 +87,5 @@
         <child link="BR_uleg_link"/>
         <limit lower="-1.2217" upper="3.14" velocity="1" effort="7"/>
-        <dynamics friction="10.0"/>
+        <dynamics friction="1.0"/>
     </joint>
     <!-- *********  BR_lleg  ********* -->
@@ -100,5 +105,5 @@
         <child link="BL_hip_link"/>
         <limit lower="-1.57" upper="1.57" velocity="1" effort="7"/>
-        <dynamics friction="10.0"/>
+        <dynamics friction="1.0"/>
     </joint>
     <!-- *********  BL_uleg  ********* -->
@@ -109,5 +114,5 @@
         <child link="BL_uleg_link"/>
         <limit lower="-1.2217" upper="3.14" velocity="1" effort="7"/>
-        <dynamics friction="10.0"/>
+        <dynamics friction="1.0"/>
     </joint>
     <!-- *********  BL_lleg  ********* -->

File: hyperdog_gazebo_sim/description/hyperdog_urdf_links.xacro (robot description, xacro)
@@ -279,3 +279,10 @@
         <xacro:inertial_left_lleg></xacro:inertial_left_lleg>
     </link>
+    <link name="imu_link">
+	  <inertial>
+		<origin xyz="0 0 0"/>
+		<mass value="0.005"/>
+		<inertia ixx="1.67e-8" ixy="0" ixz="0" iyy="1.67e-8" iyz="0" izz="1.67e-8" />
+	  </inertial>
+	</link>
 </robot>

File: hyperdog_gazebo_sim/description/physics.xacro (robot description, xacro)
@@ -62,8 +62,34 @@
     <!-- Configure foot surface -->
     <xacro:macro name="foot_surface">
-        <mu1>1</mu1>
-        <mu2>1</mu2>
-        <minDepth>0.03</minDepth>
-        <fdir1>1 1 0</fdir1>
+        <selfCollide>false</selfCollide>
+      <mu1>1.0</mu1>
+      <mu2>1.0</mu2>
+      <minDepth>0.0002</minDepth>
+      <kp>1000000.0</kp>
+      <kd>100.0</kd>
+                <gravity>true</gravity>
+                <collision name="foot_surface">
+                        <geometry>
+                                <sphere>
+                                        <!-- should be the same as surface_radius -->
+                                        <radius>0.1</radius>
+                                </sphere>
+                        </geometry>
+                <surface>
+                        <friction>
+                                <torsional>
+                                        <coefficient>10</coefficient>
+                                        <use_patch_radius>false</use_patch_radius>
+                                        <!-- should be the same as collision sphere radius -->
+                                        <surface_radius>0.1</surface_radius>
+                                        <patch_radius>0.2</patch_radius>
+                                </torsional>
+                        </friction>
+                        <contact>
+                                <poissons_ratio>0.5</poissons_ratio>
+                                <elastic_modulus>1e8</elastic_modulus>
+                        </contact>
+                </surface>
+        </collision>
     </xacro:macro>
 </robot>

Commit message: Revert "Gazebo simulation model issues fixed"

File: hyperdog_gazebo_sim/description/gazebo_ros2_control_plugin.xacro (robot description, xacro)
@@ -151,43 +151,4 @@
           <parameters>$(find hyperdog_gazebo_sim)/config/hyperdog_joint_controller.yaml</parameters>
         </plugin>
-         <plugin name="p3d_base_controller" filename="libgazebo_ros_p3d.so">
-         <ros>
-            <namespace>hyperdog</namespace>
-            <remapping>odom:=odom</remapping>
-            </ros>
-         <frame_name>map</frame_name>
-            <body_name>base_link</body_name>
-            <update_rate>200.0</update_rate>
-            <gaussian_noise>0.0</gaussian_noise>
-        <alwaysOn>true</alwaysOn>
-        <xyzOffsets>0 0 0</xyzOffsets>
-        <rpyOffsets>0 0 0</rpyOffsets>
-        </plugin>
     </gazebo>
-    <!--plugin name="imu_plugin" filename="libgazebo_ros_imu.so">
-      <alwaysOn>true</alwaysOn>
-      <body_name>imu_link</body_name>
-      <frame_name>imu_link</frame_name>
-      <topic_name>imu</topic_name>
-      <serviceName>imu_service</serviceName>
-      <gaussianNoise>0.0</gaussianNoise>
-      <updateRate>0</updateRate>
-      <imu>
-        <noise>
-          <type>gaussian</type>
-          <rate>
-            <mean>0.0</mean>
-            <stddev>2e-4</stddev>
-            <bias_mean>0.0000075</bias_mean>
-            <bias_stddev>0.0000008</bias_stddev>
-          </rate>
-          <accel>
-            <mean>0.0</mean>
-            <stddev>1.7e-2</stddev>
-            <bias_mean>0.1</bias_mean>
-            <bias_stddev>0.001</bias_stddev>
-          </accel>
-        </noise>
-      </imu>
-    </plugin-->
 </robot>

File: hyperdog_gazebo_sim/description/hyperdog_gazebo.xacro (robot description, xacro)
@@ -12,109 +12,48 @@
     <xacro:include filename="physics.xacro" />
     <gazebo reference="base_link">
-    <selfCollide>false</selfCollide>
-      <mu1 value="0.05" />
-      <mu2 value="0.05" />
         <material>Gazebo/DarkGrey  </material>
     </gazebo>
     <gazebo reference="FR_hip_link">
-    <mu1>0.2</mu1>
-    <mu2>0.2</mu2>
         <material>Gazebo/PioneerBody</material>
     </gazebo>
     <gazebo reference="FL_hip_link">
-    <mu1>0.2</mu1>
-    <mu2>0.2</mu2>
         <material>Gazebo/PioneerBody</material>
     </gazebo>
     <gazebo reference="BR_hip_link">
-    <mu1>0.2</mu1>
-    <mu2>0.2</mu2>
         <material>Gazebo/PioneerBody</material>
     </gazebo>
     <gazebo reference="BL_hip_link">
-    <mu1>0.2</mu1>
-    <mu2>0.2</mu2>
         <material>Gazebo/PioneerBody</material>
     </gazebo>
     <gazebo reference="FR_uleg_link">
-    <mu1>0.2</mu1>
-    <mu2>0.2</mu2>
         <material>Gazebo/Orange     </material>
     </gazebo>
     <gazebo reference="FL_uleg_link">
-    <mu1>0.2</mu1>
-    <mu2>0.2</mu2>
         <material>Gazebo/Orange   </material>
     </gazebo>
     <gazebo reference="BR_uleg_link">
-    <mu1>0.2</mu1>
-    <mu2>0.2</mu2>
         <material>Gazebo/Orange   </material>
     </gazebo>
     <gazebo reference="BL_uleg_link">
-    <mu1>0.2</mu1>
-    <mu2>0.2</mu2>
         <material>Gazebo/Orange </material>
     </gazebo>
     <gazebo reference="FR_lleg_link">
-    <mu1>0.2</mu1>
-    <mu2>0.2</mu2>
         <material>Gazebo/DarkYellow</material>
         <xacro:foot_surface></xacro:foot_surface>
     </gazebo>
     <gazebo reference="FL_lleg_link">
-    <mu1>0.2</mu1>
-    <mu2>0.2</mu2>
         <material>Gazebo/DarkYellow</material>
         <xacro:foot_surface></xacro:foot_surface>
     </gazebo>
     <gazebo reference="BR_lleg_link">
-    <mu1>0.2</mu1>
-    <mu2>0.2</mu2>
         <material>Gazebo/DarkYellow</material>
         <xacro:foot_surface></xacro:foot_surface>
     </gazebo>
     <gazebo reference="BL_lleg_link">
-    <mu1>0.2</mu1>
-    <mu2>0.2</mu2>
         <material>Gazebo/DarkYellow</material>
         <xacro:foot_surface></xacro:foot_surface>
     </gazebo>
-    <!--gazebo reference="FR_lleg_joint">
-    <mu1>0.1</mu1>
-    <mu2>0.1</mu2>
-    <kp>500000.0</kp>
-    <kd>10.0</kd>
-    <minDepth>0.001</minDepth>
-    <fdir1>1 0 0</fdir1>
+    <gazebo reference="FR_lleg_joint">
         <implicitSpringDamper>2</implicitSpringDamper>
-    </gazebo-->
-    <!--gazebo reference="imu_link">
-    <plugin name="imu_plugin" filename="libgazebo_ros_imu.so">
-      <alwaysOn>true</alwaysOn>
-      <bodyName>imu_link</bodyName>
-      <frameName>imu_link</frameName>
-      <topicName>imu</topicName>
-      <serviceName>imu_service</serviceName>
-      <gaussianNoise>0.0</gaussianNoise>
-      <updateRate>0</updateRate>
-      <imu>
-        <noise>
-          <type>gaussian</type>
-          <rate>
-            <mean>0.0</mean>
-            <stddev>2e-4</stddev>
-            <bias_mean>0.0000075</bias_mean>
-            <bias_stddev>0.0000008</bias_stddev>
-          </rate>
-          <accel>
-            <mean>0.0</mean>
-            <stddev>1.7e-2</stddev>
-            <bias_mean>0.1</bias_mean>
-            <bias_stddev>0.001</bias_stddev>
-          </accel>
-        </noise>
-      </imu>
-    </plugin>
-  </gazebo-->
+    </gazebo>
 </robot>

File: hyperdog_gazebo_sim/description/hyperdog_urdf_joints.xacro (robot description, xacro)
@@ -12,9 +12,4 @@
         <child link="inertial_link"/>
     </joint>
-	<joint name="imu_joint" type="fixed">
-	  <origin xyz="0 0 0" rpy="0 0 0"/>
-	  <parent link="base_link"/>
-	  <child link="imu_link"/>
-	</joint>
     <!-- *********  FR_hip  ********* -->
     <joint name="FR_hip_joint" type="revolute">
@@ -24,5 +19,5 @@
         <child link="FR_hip_link"/>
         <limit lower="-1.57" upper="1.57" velocity="1" effort="7"/>
-        <dynamics friction="1.0"/>
+        <dynamics friction="10.0"/>
     </joint>
     <!-- *********  FR_uleg  ********* -->
@@ -33,5 +28,5 @@
         <child link="FR_uleg_link"/>
         <limit lower="-1.2217" upper="3.14" velocity="1" effort="7"/>
-        <dynamics friction="1.0"/>
+        <dynamics friction="10.0"/>
     </joint>
     <!-- *********  FR_lleg  ********* -->
@@ -51,5 +46,5 @@
         <child link="FL_hip_link"/>
         <limit lower="-1.57" upper="1.57" velocity="1" effort="7"/>
-        <dynamics friction="1.0"/>
+        <dynamics friction="10.0"/>
     </joint>
     <!-- *********  FL_uleg  ********* -->
@@ -60,5 +55,5 @@
         <child link="FL_uleg_link"/>
         <limit lower="-1.2217" upper="3.14" velocity="1" effort="7"/>
-        <dynamics friction="1.0"/>
+        <dynamics friction="10.0"/>
     </joint>
     <!-- *********  FL_lleg  ********* -->
@@ -78,5 +73,5 @@
         <child link="BR_hip_link"/>
         <limit lower="-1.57" upper="1.57" velocity="1" effort="7"/>
-        <dynamics friction="1.0"/>
+        <dynamics friction="10.0"/>
     </joint>
     <!-- *********  BR_uleg  ********* -->
@@ -87,5 +82,5 @@
         <child link="BR_uleg_link"/>
         <limit lower="-1.2217" upper="3.14" velocity="1" effort="7"/>
-        <dynamics friction="1.0"/>
+        <dynamics friction="10.0"/>
     </joint>
     <!-- *********  BR_lleg  ********* -->
@@ -105,5 +100,5 @@
         <child link="BL_hip_link"/>
         <limit lower="-1.57" upper="1.57" velocity="1" effort="7"/>
-        <dynamics friction="1.0"/>
+        <dynamics friction="10.0"/>
     </joint>
     <!-- *********  BL_uleg  ********* -->
@@ -114,5 +109,5 @@
         <child link="BL_uleg_link"/>
         <limit lower="-1.2217" upper="3.14" velocity="1" effort="7"/>
-        <dynamics friction="1.0"/>
+        <dynamics friction="10.0"/>
     </joint>
     <!-- *********  BL_lleg  ********* -->

File: hyperdog_gazebo_sim/description/hyperdog_urdf_links.xacro (robot description, xacro)
@@ -279,10 +279,3 @@
         <xacro:inertial_left_lleg></xacro:inertial_left_lleg>
     </link>
-    <link name="imu_link">
-	  <inertial>
-		<origin xyz="0 0 0"/>
-		<mass value="0.005"/>
-		<inertia ixx="1.67e-8" ixy="0" ixz="0" iyy="1.67e-8" iyz="0" izz="1.67e-8" />
-	  </inertial>
-	</link>
 </robot>

File: hyperdog_gazebo_sim/description/physics.xacro (robot description, xacro)
@@ -62,34 +62,8 @@
     <!-- Configure foot surface -->
     <xacro:macro name="foot_surface">
-        <selfCollide>false</selfCollide>
-      <mu1>1.0</mu1>
-      <mu2>1.0</mu2>
-      <minDepth>0.0002</minDepth>
-      <kp>1000000.0</kp>
-      <kd>100.0</kd>
-                <gravity>true</gravity>
-                <collision name="foot_surface">
-                        <geometry>
-                                <sphere>
-                                        <!-- should be the same as surface_radius -->
-                                        <radius>0.1</radius>
-                                </sphere>
-                        </geometry>
-                <surface>
-                        <friction>
-                                <torsional>
-                                        <coefficient>10</coefficient>
-                                        <use_patch_radius>false</use_patch_radius>
-                                        <!-- should be the same as collision sphere radius -->
-                                        <surface_radius>0.1</surface_radius>
-                                        <patch_radius>0.2</patch_radius>
-                                </torsional>
-                        </friction>
-                        <contact>
-                                <poissons_ratio>0.5</poissons_ratio>
-                                <elastic_modulus>1e8</elastic_modulus>
-                        </contact>
-                </surface>
-        </collision>
+        <mu1>1</mu1>
+        <mu2>1</mu2>
+        <minDepth>0.03</minDepth>
+        <fdir1>1 1 0</fdir1>
     </xacro:macro>
 </robot>
