Commit message: 3june update

File: hyperdog_gazebo_sim/description/hyperdog_gazebo.xacro (robot description, xacro)
@@ -12,44 +12,44 @@
     <xacro:include filename="physics_include.xacro" />
     <gazebo reference="rob_link">
-        <material>Gazebo/Green</material>
+        <material>Gazebo/DarkGrey  </material>
     </gazebo>
     <gazebo reference="FR_hip_link">
-        <material>Gazebo/Blue</material>
+        <material>Gazebo/PioneerBody</material>
     </gazebo>
     <gazebo reference="FL_hip_link">
-        <material>Gazebo/Blue</material>
+        <material>Gazebo/PioneerBody</material>
     </gazebo>
     <gazebo reference="BR_hip_link">
-        <material>Gazebo/Blue</material>
+        <material>Gazebo/PioneerBody</material>
     </gazebo>
     <gazebo reference="BL_hip_link">
-        <material>Gazebo/Blue</material>
+        <material>Gazebo/PioneerBody</material>
     </gazebo>
     <gazebo reference="FR_uleg_link">
-        <material>Gazebo/Orange</material>
+        <material>Gazebo/Orange     </material>
     </gazebo>
     <gazebo reference="FL_uleg_link">
-        <material>Gazebo/Orange</material>
+        <material>Gazebo/Orange   </material>
     </gazebo>
     <gazebo reference="BR_uleg_link">
-        <material>Gazebo/Orange</material>
+        <material>Gazebo/Orange   </material>
     </gazebo>
     <gazebo reference="BL_uleg_link">
-        <material>Gazebo/Orange</material>
+        <material>Gazebo/Orange </material>
     </gazebo>
     <gazebo reference="FR_lleg_link">
-        <material>Gazebo/Red</material>
+        <material>Gazebo/DarkYellow  </material>
         <xacro:foot_surface></xacro:foot_surface>
     </gazebo>
     <gazebo reference="FL_lleg_link">
-        <material>Gazebo/Red</material>
+        <material>Gazebo/DarkYellow  </material>
         <xacro:foot_surface></xacro:foot_surface>
     </gazebo>
     <gazebo reference="BR_lleg_link">
-        <material>Gazebo/Red</material>
+        <material>Gazebo/DarkYellow  </material>
         <xacro:foot_surface></xacro:foot_surface>
     </gazebo>
     <gazebo reference="BL_lleg_link">
-        <material>Gazebo/Red</material>
+        <material>Gazebo/DarkYellow  </material>
         <xacro:foot_surface></xacro:foot_surface>
     </gazebo>

File: hyperdog_gazebo_sim/description/hyperdog_urdf_links.xacro (robot description, xacro)
@@ -182,7 +182,7 @@
                 <xacro:lleg_mesh></xacro:lleg_mesh>
             </geometry>
-            <!-- <surface>
-                <xacro:foot_surface></xacro:foot_surface>
-            </surface> -->
+            <surface>
+                <xacro:foot_surface></xacro:foot_surface>
+            </surface>
         </collision>
         <xacro:inertial_right_lleg></xacro:inertial_right_lleg>
@@ -202,4 +202,7 @@
                 <xacro:leftHip_mesh></xacro:leftHip_mesh>
             </geometry>
+            <surface>
+                <xacro:foot_surface></xacro:foot_surface>
+            </surface>
         </collision>
         <xacro:inertial_left_hip></xacro:inertial_left_hip>
@@ -219,4 +222,7 @@
                 <xacro:leftUleg_mesh></xacro:leftUleg_mesh>
             </geometry>
+            <surface>
+                <xacro:foot_surface></xacro:foot_surface>
+            </surface>
         </collision>
         <xacro:inertial_left_uleg></xacro:inertial_left_uleg>
@@ -236,7 +242,7 @@
                 <xacro:lleg_mesh></xacro:lleg_mesh>
             </geometry>
-            <!-- <surface>
-                <xacro:foot_surface></xacro:foot_surface>
-            </surface> -->
+            <surface>
+                <xacro:foot_surface></xacro:foot_surface>
+            </surface>
         </collision>
         <xacro:inertial_left_lleg></xacro:inertial_left_lleg>

File: hyperdog_gazebo_sim/description/physics_include.xacro (robot description, xacro)
@@ -28,14 +28,14 @@
         <!-- <friction>
         <mu1>10.0</mu1><mu2>10.0</mu2>
-        </friction>
+        </friction>-->
         <contact>
-            <min_depth>0.003</min_depth>
-        </contact> -->
+            <min_depth>0.001</min_depth>
+        </contact>
         <mu1>100.0</mu1>
-        <mu2>50.0</mu2>
+        <mu2>100.0</mu2>
         <kp>1e13</kp>
         <kd>1.0</kd>
-        <minDepth>0.003</minDepth>
-        <bounce_threshold>1</bounce_threshold>
+        <minDepth>0.001</minDepth>
+        <bounce_threshold>10000000</bounce_threshold>
         <maxVel>0.1</maxVel>
         <fdir1>0 0 0</fdir1>

Commit message: updated ign sim urdfs

File: hyperdog_gazebo_sim/description/hyperdog_gazebo.xacro (robot description, xacro)
@@ -10,6 +10,6 @@
     Instead, we need to add gazebo tags for our links that refer to Gazebo materials
 -->
-    <xacro:include filename="physics_include.xacro" />
-    <gazebo reference="rob_link">
+    <xacro:include filename="physics.xacro" />
+    <gazebo reference="base_link">
         <material>Gazebo/DarkGrey  </material>
     </gazebo>
@@ -39,21 +39,21 @@
     </gazebo>
     <gazebo reference="FR_lleg_link">
-        <material>Gazebo/DarkYellow  </material>
+        <material>Gazebo/DarkYellow</material>
         <xacro:foot_surface></xacro:foot_surface>
     </gazebo>
     <gazebo reference="FL_lleg_link">
-        <material>Gazebo/DarkYellow  </material>
+        <material>Gazebo/DarkYellow</material>
         <xacro:foot_surface></xacro:foot_surface>
     </gazebo>
     <gazebo reference="BR_lleg_link">
-        <material>Gazebo/DarkYellow  </material>
+        <material>Gazebo/DarkYellow</material>
         <xacro:foot_surface></xacro:foot_surface>
     </gazebo>
     <gazebo reference="BL_lleg_link">
-        <material>Gazebo/DarkYellow  </material>
+        <material>Gazebo/DarkYellow</material>
         <xacro:foot_surface></xacro:foot_surface>
     </gazebo>
-    <gazebo reference=" FR_lleg_joint">
-        <implicitSpringDamper>1</implicitSpringDamper>
+    <gazebo reference="FR_lleg_joint">
+        <implicitSpringDamper>2</implicitSpringDamper>
     </gazebo>
 </robot>

File: hyperdog_gazebo_sim/description/hyperdog_urdf_joints.xacro (robot description, xacro)
@@ -7,9 +7,14 @@
                     <xacro:include filename="hyperdog_urdf_joints.xacro" />
     _____________________________________________________________________ -->
+    <!-- ******** Inertial ********** -->
+    <joint name="inertial_joint" type="fixed">
+        <parent link="base_link"/>
+        <child link="inertial_link"/>
+    </joint>
     <!-- *********  FR_hip  ********* -->
     <joint name="FR_hip_joint" type="revolute">
         <axis xyz="-1 0 0"/>
         <origin xyz="0.175 -0.066 0" rpy="0 0 0"/>
-        <parent link="rob_link"/>
+        <parent link="base_link"/>
         <child link="FR_hip_link"/>
         <limit lower="-1.57" upper="1.57" velocity="1" effort="7"/>
@@ -38,5 +43,5 @@
         <axis xyz="1 0 0"/>
         <origin xyz="0.175 0.066 0" rpy="0 0 0"/>
-        <parent link="rob_link"/>
+        <parent link="base_link"/>
         <child link="FL_hip_link"/>
         <limit lower="-1.57" upper="1.57" velocity="1" effort="7"/>
@@ -65,5 +70,5 @@
         <axis xyz="-1 0 0"/>
         <origin xyz="-0.175 -0.066 0" rpy="0 0 0"/>
-        <parent link="rob_link"/>
+        <parent link="base_link"/>
         <child link="BR_hip_link"/>
         <limit lower="-1.57" upper="1.57" velocity="1" effort="7"/>
@@ -92,5 +97,5 @@
         <axis xyz="1 0 0"/>
         <origin xyz="-0.175 0.066 0" rpy="0 0 0"/>
-        <parent link="rob_link"/>
+        <parent link="base_link"/>
         <child link="BL_hip_link"/>
         <limit lower="-1.57" upper="1.57" velocity="1" effort="7"/>

File: hyperdog_gazebo_sim/description/hyperdog_urdf_links.xacro (robot description, xacro)
@@ -2,4 +2,6 @@
 <robot xmlns:xacro="http://www.ros.org/wiki/xacro">
 <!--
+    * Autor: nipun.dhananjaya@gmail.com
+    * Date:  13.03.2023
     _____________________________________________________________________
         include this file into: /description/hyperdog.urdf.xacro
@@ -7,6 +9,30 @@
                     <xacro:include filename="hyperdog_urdf_links.xacro" />
     _____________________________________________________________________ -->
-    <xacro:include filename="physics_include.xacro" />
-    <link name="rob_link">
+    <xacro:include filename="physics.xacro" />
+    <!-- load meshes -->
+    <xacro:macro name="body_mesh">
+        <mesh filename="file://$(find hyperdog_gazebo_sim)/meshes/body.stl" scale="0.001 0.001 0.001"/>
+    </xacro:macro>
+    <xacro:macro name="rightHip_mesh">
+        <mesh filename="file://$(find hyperdog_gazebo_sim)/meshes/RIGHT_HIP.stl" scale="0.001 0.001 0.001"/>
+    </xacro:macro>
+    <xacro:macro name="leftHip_mesh">
+        <mesh filename="file://$(find hyperdog_gazebo_sim)/meshes/LEFT_HIP.stl" scale="0.001 0.001 0.001"/>
+    </xacro:macro>
+    <xacro:macro name="rightUleg_mesh">
+        <mesh filename="file://$(find hyperdog_gazebo_sim)/meshes/RIGHT_ULEG.stl" scale="0.001 0.001 0.001"/>
+    </xacro:macro>
+    <xacro:macro name="leftUleg_mesh">
+        <mesh filename="file://$(find hyperdog_gazebo_sim)/meshes/LEFT_ULEG.stl" scale="0.001 0.001 0.001"/>
+    </xacro:macro>
+    <xacro:macro name="lleg_mesh">
+        <mesh filename="file://$(find hyperdog_gazebo_sim)/meshes/LLEG.stl" scale="0.001 0.001 0.001"/>
+    </xacro:macro>
+    <!-- *********** Inertial link *********** -->
+    <link name="inertial_link">
+        <xacro:inertial_body></xacro:inertial_body>
+    </link>
+    <!-- *********** base link *********** -->
+    <link name="base_link">
         <visual>
             <origin xyz="0 0 0" rpy="0 0 0"/>
@@ -24,5 +50,4 @@
             </geometry>
         </collision>
-        <xacro:inertial_body></xacro:inertial_body>
     </link>
     <!-- *********** FR_hip *********** -->
@@ -80,7 +105,4 @@
                 <xacro:lleg_mesh></xacro:lleg_mesh>
             </geometry>
-            <!-- <surface>
-                <xacro:foot_surface></xacro:foot_surface>
-            </surface> -->
         </collision>
         <xacro:inertial_right_lleg></xacro:inertial_right_lleg>
@@ -88,5 +110,5 @@
     <!-- *********** FL_hip ********** -->
     <link name="FL_hip_link">
-        <visual>curve
+        <visual>
             <origin xyz="0 0 0" rpy="0 0 0"/>
             <geometry>
@@ -140,7 +162,4 @@
                 <xacro:lleg_mesh></xacro:lleg_mesh>
             </geometry>
-            <!-- <surface>
-                <xacro:foot_surface></xacro:foot_surface>
-            </surface> -->
         </collision>
         <xacro:inertial_left_lleg></xacro:inertial_left_lleg>
@@ -200,7 +219,4 @@
                 <xacro:lleg_mesh></xacro:lleg_mesh>
             </geometry>
-            <surface>
-                <xacro:foot_surface></xacro:foot_surface>
-            </surface>
         </collision>
         <xacro:inertial_right_lleg></xacro:inertial_right_lleg>
@@ -222,7 +238,4 @@
                 <xacro:leftHip_mesh></xacro:leftHip_mesh>
             </geometry>
-            <surface>
-                <xacro:foot_surface></xacro:foot_surface>
-            </surface>
         </collision>
         <xacro:inertial_left_hip></xacro:inertial_left_hip>
@@ -244,7 +257,4 @@
                 <xacro:leftUleg_mesh></xacro:leftUleg_mesh>
             </geometry>
-            <surface>
-                <xacro:foot_surface></xacro:foot_surface>
-            </surface>
         </collision>
         <xacro:inertial_left_uleg></xacro:inertial_left_uleg>
@@ -266,7 +276,4 @@
                 <xacro:lleg_mesh></xacro:lleg_mesh>
             </geometry>
-            <surface>
-                <xacro:foot_surface></xacro:foot_surface>
-            </surface>
         </collision>
         <xacro:inertial_left_lleg></xacro:inertial_left_lleg>

File: hyperdog_gazebo_sim/description/physics.xacro (robot description, xacro)
@@ -1,44 +1,4 @@
 <?xml version="1.0"?>
 <robot xmlns:xacro="http://www.ros.org/wiki/xacro" >
-    <!-- Include meshes -->
-    <xacro:macro name="body_mesh">
-        <mesh filename="file://$(find hyperdog_gazebo_sim)/meshes/body.stl" scale="0.001 0.001 0.001"/>
-    </xacro:macro>
-    <xacro:macro name="rightHip_mesh">
-        <mesh filename="file://$(find hyperdog_gazebo_sim)/meshes/RIGHT_HIP.stl" scale="0.001 0.001 0.001"/>
-    </xacro:macro>
-    <xacro:macro name="leftHip_mesh">
-        <mesh filename="file://$(find hyperdog_gazebo_sim)/meshes/LEFT_HIP.stl" scale="0.001 0.001 0.001"/>
-    </xacro:macro>
-    <xacro:macro name="rightUleg_mesh">
-        <mesh filename="file://$(find hyperdog_gazebo_sim)/meshes/RIGHT_ULEG.stl" scale="0.001 0.001 0.001"/>
-    </xacro:macro>
-    <xacro:macro name="leftUleg_mesh">
-        <mesh filename="file://$(find hyperdog_gazebo_sim)/meshes/LEFT_ULEG.stl" scale="0.001 0.001 0.001"/>
-    </xacro:macro>
-    <xacro:macro name="lleg_mesh">
-        <mesh filename="file://$(find hyperdog_gazebo_sim)/meshes/LLEG.stl" scale="0.001 0.001 0.001"/>
-    </xacro:macro>
-    <!-- Configure joint dynamics -->
-    <xacro:macro name="lleg_jointDynamics">
-        <dynamics damping="1.0" friction="1000.0"/>
-    </xacro:macro>
-    <!-- Configure foot surface -->
-    <xacro:macro name="foot_surface">
-        <!-- <friction>
-        <mu1>10.0</mu1><mu2>10.0</mu2>
-        </friction>-->
-        <contact>
-            <min_depth>0.001</min_depth>
-        </contact>
-        <mu1>100.0</mu1>
-        <mu2>100.0</mu2>
-        <kp>1e13</kp>
-        <kd>1.0</kd>
-        <minDepth>0.001</minDepth>
-        <bounce_threshold>10000000</bounce_threshold>
-        <maxVel>0.1</maxVel>
-        <fdir1>0 0 0</fdir1>
-    </xacro:macro>
     <!-- configure inertia -->
     <!--  BODY -->
@@ -95,3 +55,15 @@
         </inertial>
     </xacro:macro>
+    <!-- ************************************************************************************************** -->
+    <!-- Configure joint dynamics -->
+    <xacro:macro name="lleg_jointDynamics">
+        <dynamics damping="1.0" friction="1000.0"/>
+    </xacro:macro>
+    <!-- Configure foot surface -->
+    <xacro:macro name="foot_surface">
+        <mu1>1</mu1>
+        <mu2>1</mu2>
+        <minDepth>0.03</minDepth>
+        <fdir1>1 1 0</fdir1>
+    </xacro:macro>
 </robot>

File: hyperdog_ign_sim/xacros/gazebo_ros2_control_plugin.xacro (robot description, xacro)
@@ -146,7 +146,7 @@
         </joint>
     </ros2_control>
-    <!--  CONFIGURE THE GAZEBO PLUGIN Joint State Publisher-->
+    <!--  CONFIGURE THE GAZEBO PLUGIN -->
     <gazebo>
-        <plugin filename="libign_ros2_control-system" name="ign_ros2_control::IgnitionROS2ControlPlugin">
+        <plugin filename="ign_ros2_control-system" name="ign_ros2_control::IgnitionROS2ControlPlugin">
           <parameters>$(find hyperdog_ign_sim)/config/hyperdog_joint_controller.yaml</parameters>
         </plugin>

File: hyperdog_ign_sim/xacros/hyperdog.urdf.xacro (robot description, xacro)
@@ -2,9 +2,9 @@
 <robot xmlns:xacro="http://www.ros.org/wiki/xacro"  name="hyperdog">
     <!-- ***************  CONFIGURE ROBOT"S LINKS  *******************-->
-    <xacro:include filename="$(find hyperdog_ign_sim)/xacros/hyperdog_urdf_links.xacro"/>
+    <xacro:include filename="$(find hyperdog_ign_sim)/xacros/hyperdog_urdf_links.xacro" />
     <!-- ***************  CONFIGURE ROBOT"S JOINTS  *******************-->
-    <xacro:include filename="$(find hyperdog_ign_sim)/xacros/hyperdog_urdf_joints.xacro"/>
+    <xacro:include filename="$(find hyperdog_ign_sim)/xacros/hyperdog_urdf_joints.xacro" />
     <!-- ****************   INCLUDES OTHER FILES  ******************* -->
-    <xacro:include filename="$(find hyperdog_ign_sim)/xacros/gazebo_ros2_control_plugin.xacro"/>
-    <xacro:include filename="$(find hyperdog_ign_sim)/xacros/hyperdog_gazebo.xacro"/>
+    <xacro:include filename="$(find hyperdog_ign_sim)/xacros/gazebo_ros2_control_plugin.xacro" />
+    <!-- <xacro:include filename="$(find hyperdog_ign_sim)/xacros/hyperdog_gazebo.xacro" /> -->
 </robot>
