Commit message: updated ign sim urdfs

File: hyperdog_ign_sim/xacros/hyperdog_urdf_links.xacro (robot description, xacro)
@@ -2,4 +2,6 @@
 <robot xmlns:xacro="http://www.ros.org/wiki/xacro">
 <!--
+    * Autor: nipun.dhananjaya@gmail.com
+    * Date:  13.03.2023
     _____________________________________________________________________
         include this file into: /description/hyperdog.urdf.xacro
@@ -7,10 +9,31 @@
                     <xacro:include filename="hyperdog_urdf_links.xacro" />
     _____________________________________________________________________ -->
-    <xacro:include filename="physics_include.xacro" />
-    <link name="rob_link">
-        <must_be_base_link>true</must_be_base_link>
-        <pose>0 0 0 0 0 0</pose>
+    <xacro:include filename="physics.xacro" />
+    <!-- load meshes -->
+    <xacro:macro name="body_mesh">
+        <mesh filename="file://$(find hyperdog_ign_sim)/models/hyperdog/meshes/body.stl" scale="0.001 0.001 0.001"/>
+    </xacro:macro>
+    <xacro:macro name="rightHip_mesh">
+        <mesh filename="file://$(find hyperdog_ign_sim)/models/hyperdog/meshes/RIGHT_HIP.stl" scale="0.001 0.001 0.001"/>
+    </xacro:macro>
+    <xacro:macro name="leftHip_mesh">
+        <mesh filename="file://$(find hyperdog_ign_sim)/models/hyperdog/meshes/LEFT_HIP.stl" scale="0.001 0.001 0.001"/>
+    </xacro:macro>
+    <xacro:macro name="rightUleg_mesh">
+        <mesh filename="file://$(find hyperdog_ign_sim)/models/hyperdog/meshes/RIGHT_ULEG.stl" scale="0.001 0.001 0.001"/>
+    </xacro:macro>
+    <xacro:macro name="leftUleg_mesh">
+        <mesh filename="file://$(find hyperdog_ign_sim)/models/hyperdog/meshes/LEFT_ULEG.stl" scale="0.001 0.001 0.001"/>
+    </xacro:macro>
+    <xacro:macro name="lleg_mesh">
+        <mesh filename="file://$(find hyperdog_ign_sim)/models/hyperdog/meshes/LLEG.stl" scale="0.001 0.001 0.001"/>
+    </xacro:macro>
+    <!-- *********** Inertial link *********** -->
+    <link name="inertial_link">
         <xacro:inertial_body></xacro:inertial_body>
-        <visual name='body'>
+    </link>
+    <!-- *********** base link *********** -->
+    <link name="base_link">
+        <visual>
             <geometry>
                 <xacro:body_mesh></xacro:body_mesh>
@@ -19,256 +42,214 @@
                 <color rgba="0.2 1 0.2 1"/>
             </material>
-          </visual>
-          <collision name='collision'>
+        </visual>
+        <collision>
             <geometry>
                 <xacro:body_mesh></xacro:body_mesh>
             </geometry>
-          </collision>
+        </collision>
     </link>
     <!-- *********** FR_hip *********** -->
     <link name="FR_hip_link">
         <visual>
-            <origin xyz="0 0 0" rpy="0 0 0"/>
-            <geometry>
-                <xacro:rightHip_mesh></xacro:rightHip_mesh>
-            </geometry>
-            <material name="red">
-                <color rgba="0.8 0.2 0.2 1"/>
-            </material>
-        </visual>
-        <collision>
-            <origin xyz="0 0 0" rpy="0 0 0"/>
-            <geometry>
-                <xacro:rightHip_mesh></xacro:rightHip_mesh>
-            </geometry>
-        </collision>
-        <!-- <xacro:inertial_right_hip></xacro:inertial_right_hip> -->
+            <geometry>
+                <xacro:rightHip_mesh></xacro:rightHip_mesh>
+            </geometry>
+            <material name="red">
+                <color rgba="0.8 0.2 0.2 1"/>
+            </material>
+        </visual>
+        <collision>
+            <geometry>
+                <xacro:rightHip_mesh></xacro:rightHip_mesh>
+            </geometry>
+        </collision>
+        <xacro:inertial_right_hip></xacro:inertial_right_hip>
     </link>
     <!-- *********** FR_uleg ********** -->
     <link name="FR_uleg_link">
         <visual>
-            <origin xyz="0 0 0" rpy="0 0 0"/>
-            <geometry>
-                <xacro:rightUleg_mesh></xacro:rightUleg_mesh>
-            </geometry>
-            <material name="orange">
-                <color rgba="0.8 0.5 0.8 1"/>
-            </material>
-        </visual>
-        <collision>
-            <origin xyz="0 0 0" rpy="0 0 0"/>
-            <geometry>
-                <xacro:rightUleg_mesh></xacro:rightUleg_mesh>
-            </geometry>
-        </collision>
-        <!-- <xacro:inertial_right_uleg></xacro:inertial_right_uleg> -->
+            <geometry>
+                <xacro:rightUleg_mesh></xacro:rightUleg_mesh>
+            </geometry>
+            <material name="orange">
+                <color rgba="0.8 0.5 0.8 1"/>
+            </material>
+        </visual>
+        <collision>
+            <geometry>
+                <xacro:rightUleg_mesh></xacro:rightUleg_mesh>
+            </geometry>
+        </collision>
+        <xacro:inertial_right_uleg></xacro:inertial_right_uleg>
     </link>
     <!-- *********** FR_lleg ********** -->
     <link name="FR_lleg_link">
         <visual>
-            <origin xyz="0 0 0" rpy="0 0 0"/>
-            <geometry>
-                <xacro:lleg_mesh></xacro:lleg_mesh>
-            </geometry>
-            <material name="yellow">
-                <color rgba="0.8 1.0 0.1 1"/>
-            </material>
-        </visual>
-        <collision>
-            <origin xyz="0 0 0" rpy="0 0 0"/>
-            <geometry>
-                <xacro:lleg_mesh></xacro:lleg_mesh>
-            </geometry>
-            <!-- <surface>
-                <xacro:foot_surface></xacro:foot_surface>
-            </surface> -->
-        </collision>
-        <!-- <xacro:inertial_right_lleg></xacro:inertial_right_lleg> -->
+            <geometry>
+                <xacro:lleg_mesh></xacro:lleg_mesh>
+            </geometry>
+            <material name="yellow">
+                <color rgba="0.8 1.0 0.1 1"/>
+            </material>
+        </visual>
+        <collision>
+            <geometry>
+                <xacro:lleg_mesh></xacro:lleg_mesh>
+            </geometry>
+        </collision>
+        <xacro:inertial_right_lleg></xacro:inertial_right_lleg>
     </link>
     <!-- *********** FL_hip ********** -->
     <link name="FL_hip_link">
-        <visual>curve
-            <origin xyz="0 0 0" rpy="0 0 0"/>
-            <geometry>
-                <xacro:leftHip_mesh></xacro:leftHip_mesh>
-            </geometry>
-            <material name="red">
-                <color rgba="0.8 0.2 0.2 1"/>
-            </material>
-        </visual>
-        <collision>
-            <origin xyz="0 0 0" rpy="0 0 0"/>
-            <geometry>
-                <xacro:leftHip_mesh></xacro:leftHip_mesh>
-            </geometry>
-        </collision>
-        <!-- <xacro:inertial_left_hip></xacro:inertial_left_hip> -->
+        <visual>
+            <geometry>
+                <xacro:leftHip_mesh></xacro:leftHip_mesh>
+            </geometry>
+            <material name="red">
+                <color rgba="0.8 0.2 0.2 1"/>
+            </material>
+        </visual>
+        <collision>
+            <geometry>
+                <xacro:leftHip_mesh></xacro:leftHip_mesh>
+            </geometry>
+        </collision>
+        <xacro:inertial_left_hip></xacro:inertial_left_hip>
     </link>
     <!-- *********** FL_uleg ********** -->
     <link name="FL_uleg_link">
         <visual>
-            <origin xyz="0 0 0" rpy="0 0 0"/>
-            <geometry>
-                <xacro:leftUleg_mesh></xacro:leftUleg_mesh>
-            </geometry>
-            <material name="orange">
-                <color rgba="0.8 0.5 0.8 1"/>
-            </material>
-        </visual>
-        <collision>
-            <origin xyz="0 0 0" rpy="0 0 0"/>
-            <geometry>
-                <xacro:leftUleg_mesh></xacro:leftUleg_mesh>
-            </geometry>
-        </collision>
-        <!-- <xacro:inertial_left_uleg></xacro:inertial_left_uleg> -->
+            <geometry>
+                <xacro:leftUleg_mesh></xacro:leftUleg_mesh>
+            </geometry>
+            <material name="orange">
+                <color rgba="0.8 0.5 0.8 1"/>
+            </material>
+        </visual>
+        <collision>
+            <geometry>
+                <xacro:leftUleg_mesh></xacro:leftUleg_mesh>
+            </geometry>
+        </collision>
+        <xacro:inertial_left_uleg></xacro:inertial_left_uleg>
     </link>
     <!-- *********** FL_lleg ********** -->
     <link name="FL_lleg_link">
         <visual>
-            <origin xyz="0 0 0" rpy="0 0 0"/>
-            <geometry>
-                <xacro:lleg_mesh></xacro:lleg_mesh>
-            </geometry>
-            <material name="yellow">
-                <color rgba="0.8 1.0 0.1 1"/>
-            </material>
-        </visual>
-        <collision>
-            <origin xyz="0 0 0" rpy="0 0 0"/>
-            <geometry>
-                <xacro:lleg_mesh></xacro:lleg_mesh>
-            </geometry>
-            <!-- <surface>
-                <xacro:foot_surface></xacro:foot_surface>
-            </surface> -->
-        </collision>
-        <!-- <xacro:inertial_left_lleg></xacro:inertial_left_lleg> -->
+            <geometry>
+                <xacro:lleg_mesh></xacro:lleg_mesh>
+            </geometry>
+            <material name="yellow">
+                <color rgba="0.8 1.0 0.1 1"/>
+            </material>
+        </visual>
+        <collision>
+            <geometry>
+                <xacro:lleg_mesh></xacro:lleg_mesh>
+            </geometry>
+        </collision>
+        <xacro:inertial_left_lleg></xacro:inertial_left_lleg>
     </link>
     <!-- *********** BR_hip ********** -->
     <link name="BR_hip_link">
         <visual>
-            <origin xyz="0 0 0" rpy="0 0 0"/>
-            <geometry>
-                <xacro:rightHip_mesh></xacro:rightHip_mesh>
-            </geometry>
-            <material name="red">
-                <color rgba="0.8 0.2 0.2 1"/>
-            </material>
-        </visual>
-        <collision>
-            <origin xyz="0 0 0" rpy="0 0 0"/>
-            <geometry>
-                <xacro:rightHip_mesh></xacro:rightHip_mesh>
-            </geometry>
-        </collision>
-        <!-- <xacro:inertial_right_hip></xacro:inertial_right_hip> -->
+            <geometry>
+                <xacro:rightHip_mesh></xacro:rightHip_mesh>
+            </geometry>
+            <material name="red">
+                <color rgba="0.8 0.2 0.2 1"/>
+            </material>
+        </visual>
+        <collision>
+            <geometry>
+                <xacro:rightHip_mesh></xacro:rightHip_mesh>
+            </geometry>
+        </collision>
+        <xacro:inertial_right_hip></xacro:inertial_right_hip>
     </link>
     <!-- *********** BR_uleg ********** -->
     <link name="BR_uleg_link">
         <visual>
-            <origin xyz="0 0 0" rpy="0 0 0"/>
-            <geometry>
-                <xacro:rightUleg_mesh></xacro:rightUleg_mesh>
-            </geometry>
-            <material name="orange">
-                <color rgba="0.8 0.5 0.8 1"/>
-            </material>
-        </visual>
-        <collision>
-            <origin xyz="0 0 0" rpy="0 0 0"/>
-            <geometry>
-                <xacro:rightUleg_mesh></xacro:rightUleg_mesh>
-            </geometry>
-        </collision>
-        <!-- <xacro:inertial_right_uleg></xacro:inertial_right_uleg> -->
+            <geometry>
+                <xacro:rightUleg_mesh></xacro:rightUleg_mesh>
+            </geometry>
+            <material name="orange">
+                <color rgba="0.8 0.5 0.8 1"/>
+            </material>
+        </visual>
+        <collision>
+            <geometry>
+                <xacro:rightUleg_mesh></xacro:rightUleg_mesh>
+            </geometry>
+        </collision>
+        <xacro:inertial_right_uleg></xacro:inertial_right_uleg>
     </link>
     <!-- *********** BR_lleg ********** -->
     <link name="BR_lleg_link">
         <visual>
-            <origin xyz="0 0 0" rpy="0 0 0"/>
-            <geometry>
-                <xacro:lleg_mesh></xacro:lleg_mesh>
-            </geometry>
-            <material name="yellow">
-                <color rgba="0.8 1.0 0.1 1"/>
-            </material>
-        </visual>
-        <collision>
-            <origin xyz="0 0 0" rpy="0 0 0"/>
-            <geometry>
-                <xacro:lleg_mesh></xacro:lleg_mesh>
-            </geometry>
-            <surface>
-                <xacro:foot_surface></xacro:foot_surface>
-            </surface>
-        </collision>
-        <!-- <xacro:inertial_right_lleg></xacro:inertial_right_lleg> -->
+            <geometry>
+                <xacro:lleg_mesh></xacro:lleg_mesh>
+            </geometry>
+            <material name="yellow">
+                <color rgba="0.8 1.0 0.1 1"/>
+            </material>
+        </visual>
+        <collision>
+            <geometry>
+                <xacro:lleg_mesh></xacro:lleg_mesh>
+            </geometry>
+        </collision>
+        <xacro:inertial_right_lleg></xacro:inertial_right_lleg>
     </link>
     <!-- *********** BL_hip ********** -->
     <link name="BL_hip_link">
         <visual>
-            <origin xyz="0 0 0" rpy="0 0 0"/>
-            <geometry>
-                <xacro:leftHip_mesh></xacro:leftHip_mesh>
-            </geometry>
-            <material name="red">
-                <color rgba="0.8 0.2 0.2 1"/>
-            </material>
-        </visual>
-        <collision>
-            <origin xyz="0 0 0" rpy="0 0 0"/>
-            <geometry>
-                <xacro:leftHip_mesh></xacro:leftHip_mesh>
-            </geometry>
-            <surface>
-                <xacro:foot_surface></xacro:foot_surface>
-            </surface>
-        </collision>
-        <!-- <xacro:inertial_left_hip></xacro:inertial_left_hip> -->
+            <geometry>
+                <xacro:leftHip_mesh></xacro:leftHip_mesh>
+            </geometry>
+            <material name="red">
+                <color rgba="0.8 0.2 0.2 1"/>
+            </material>
+        </visual>
+        <collision>
+            <geometry>
+                <xacro:leftHip_mesh></xacro:leftHip_mesh>
+            </geometry>
+        </collision>
+        <xacro:inertial_left_hip></xacro:inertial_left_hip>
     </link>
     <!-- *********** BL_uleg ********** -->
     <link name="BL_uleg_link">
         <visual>
-            <origin xyz="0 0 0" rpy="0 0 0"/>
-            <geometry>
-                <xacro:leftUleg_mesh></xacro:leftUleg_mesh>
-            </geometry>
-            <material name="orange">
-                <color rgba="0.8 0.5 0.8 1"/>
-            </material>
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