Commit message: updated urdf. added foots

File: hyperdog_gazebo_sim/description/hyperdog_gazebo.xacro (robot description, xacro)
@@ -13,47 +13,116 @@
     <gazebo reference="base_link">
         <material>Gazebo/DarkGrey  </material>
+        <mu1>0.2</mu1>
+        <mu2>0.2</mu2>
+        <kp value="1000000.0"/>
+        <kd value="1.0"/>
     </gazebo>
     <gazebo reference="FR_hip_link">
+        <mu1>0.2</mu1>
+        <mu2>0.2</mu2>
         <material>Gazebo/PioneerBody</material>
     </gazebo>
     <gazebo reference="FL_hip_link">
+        <mu1>0.2</mu1>
+        <mu2>0.2</mu2>
         <material>Gazebo/PioneerBody</material>
     </gazebo>
     <gazebo reference="BR_hip_link">
+        <mu1>0.2</mu1>
+        <mu2>0.2</mu2>
         <material>Gazebo/PioneerBody</material>
     </gazebo>
     <gazebo reference="BL_hip_link">
+        <mu1>0.2</mu1>
+        <mu2>0.2</mu2>
         <material>Gazebo/PioneerBody</material>
     </gazebo>
     <gazebo reference="FR_uleg_link">
-        <material>Gazebo/Orange     </material>
+        <mu1>0.2</mu1>
+        <mu2>0.2</mu2>
+        <self_collide>1</self_collide>
+        <kp value="1000000.0"/>
+        <kd value="1.0"/>
+        <material>Gazebo/Orange</material>
     </gazebo>
     <gazebo reference="FL_uleg_link">
+        <mu1>0.2</mu1>
+        <mu2>0.2</mu2>
+        <self_collide>1</self_collide>
+        <kp value="1000000.0"/>
+        <kd value="1.0"/>
         <material>Gazebo/Orange   </material>
     </gazebo>
     <gazebo reference="BR_uleg_link">
+        <mu1>0.2</mu1>
+        <mu2>0.2</mu2>
+        <self_collide>1</self_collide>
+        <kp value="1000000.0"/>
+        <kd value="1.0"/>
         <material>Gazebo/Orange   </material>
     </gazebo>
     <gazebo reference="BL_uleg_link">
+        <mu1>0.2</mu1>
+        <mu2>0.2</mu2>
+        <self_collide>1</self_collide>
+        <kp value="1000000.0"/>
+        <kd value="1.0"/>
         <material>Gazebo/Orange </material>
     </gazebo>
     <gazebo reference="FR_lleg_link">
         <material>Gazebo/DarkYellow</material>
-        <xacro:foot_surface></xacro:foot_surface>
+        <mu1>0.2</mu1>
+        <mu2>0.2</mu2>
+        <self_collide>1</self_collide>
     </gazebo>
     <gazebo reference="FL_lleg_link">
         <material>Gazebo/DarkYellow</material>
-        <xacro:foot_surface></xacro:foot_surface>
+        <mu1>0.2</mu1>
+        <mu2>0.2</mu2>
+        <self_collide>1</self_collide>
     </gazebo>
     <gazebo reference="BR_lleg_link">
         <material>Gazebo/DarkYellow</material>
-        <xacro:foot_surface></xacro:foot_surface>
+        <mu1>0.2</mu1>
+        <mu2>0.2</mu2>
+        <self_collide>1</self_collide>
     </gazebo>
     <gazebo reference="BL_lleg_link">
         <material>Gazebo/DarkYellow</material>
-        <xacro:foot_surface></xacro:foot_surface>
+        <mu1>0.2</mu1>
+        <mu2>0.2</mu2>
+        <self_collide>1</self_collide>
     </gazebo>
-    <gazebo reference="FR_lleg_joint">
-        <implicitSpringDamper>2</implicitSpringDamper>
+    <gazebo reference="FR_foot">
+        <material>Gazebo/DarkGrey</material>
+        <mu1>0.6</mu1>
+        <mu2>0.6</mu2>
+        <self_collide>1</self_collide>
+        <kp value="1000000.0"/>
+        <kd value="1.0"/>
+    </gazebo>
+    <gazebo reference="FL_foot">
+        <material>Gazebo/DarkGrey</material>
+        <mu1>0.6</mu1>
+        <mu2>0.6</mu2>
+        <self_collide>1</self_collide>
+        <kp value="1000000.0"/>
+        <kd value="1.0"/>
+    </gazebo>
+    <gazebo reference="BL_foot">
+        <material>Gazebo/DarkGrey</material>
+        <mu1>0.6</mu1>
+        <mu2>0.6</mu2>
+        <self_collide>1</self_collide>
+        <kp value="1000000.0"/>
+        <kd value="1.0"/>
+    </gazebo>
+    <gazebo reference="BR_foot">
+        <material>Gazebo/DarkGrey</material>
+        <mu1>0.6</mu1>
+        <mu2>0.6</mu2>
+        <self_collide>1</self_collide>
+        <kp value="1000000.0"/>
+        <kd value="1.0"/>
     </gazebo>
 </robot>

File: hyperdog_gazebo_sim/description/hyperdog_urdf_joints.xacro (robot description, xacro)
@@ -18,6 +18,6 @@
         <parent link="base_link"/>
         <child link="FR_hip_link"/>
-        <limit lower="-1.57" upper="1.57" velocity="1" effort="7"/>
-        <dynamics friction="10.0"/>
+        <limit lower="-1.57" upper="1.57" velocity="21" effort="7"/>
+        <dynamics damping="0.01" friction="0.2"/>
     </joint>
     <!-- *********  FR_uleg  ********* -->
@@ -28,5 +28,5 @@
         <child link="FR_uleg_link"/>
         <limit lower="-1.2217" upper="3.14" velocity="1" effort="7"/>
-        <dynamics friction="10.0"/>
+        <dynamics damping="0.01" friction="0.2"/>
     </joint>
     <!-- *********  FR_lleg  ********* -->
@@ -37,6 +37,12 @@
         <child link="FR_lleg_link"/>
         <limit lower="-1.57" upper="2.618" velocity="1" effort="7"/>
-        <xacro:lleg_jointDynamics></xacro:lleg_jointDynamics>
+        <dynamics damping="0.01" friction="0.2"/>
     </joint>
+     <!-- *********  FR_FOOT  ********* -->
+     <joint name="FR_foot_fixed" type="fixed">
+        <origin rpy="0 0 0" xyz="0.14 0 0"/>
+        <parent link="FR_lleg_link"/>
+        <child link="FR_foot"/>
+      </joint>
     <!-- *********  FL_hip  ********* -->
     <joint name="FL_hip_joint" type="revolute">
@@ -46,5 +52,5 @@
         <child link="FL_hip_link"/>
         <limit lower="-1.57" upper="1.57" velocity="1" effort="7"/>
-        <dynamics friction="10.0"/>
+        <dynamics damping="0.01" friction="0.2"/>
     </joint>
     <!-- *********  FL_uleg  ********* -->
@@ -55,5 +61,5 @@
         <child link="FL_uleg_link"/>
         <limit lower="-1.2217" upper="3.14" velocity="1" effort="7"/>
-        <dynamics friction="10.0"/>
+        <dynamics damping="0.01" friction="0.2"/>
     </joint>
     <!-- *********  FL_lleg  ********* -->
@@ -64,6 +70,12 @@
         <child link="FL_lleg_link"/>
         <limit lower="-1.57" upper="2.618" velocity="1" effort="7"/>
-        <xacro:lleg_jointDynamics></xacro:lleg_jointDynamics>
+        <dynamics damping="0.01" friction="0.2"/>
     </joint>
+     <!-- *********  FL_FOOT  ********* -->
+     <joint name="FL_foot_fixed" type="fixed">
+        <origin rpy="0 0 0" xyz="0.14 0 0"/>
+        <parent link="FL_lleg_link"/>
+        <child link="FL_foot"/>
+      </joint>
     <!-- *********  BR_hip  ********* -->
     <joint name="BR_hip_joint" type="revolute">
@@ -73,5 +85,5 @@
         <child link="BR_hip_link"/>
         <limit lower="-1.57" upper="1.57" velocity="1" effort="7"/>
-        <dynamics friction="10.0"/>
+        <dynamics damping="0.01" friction="0.2"/>
     </joint>
     <!-- *********  BR_uleg  ********* -->
@@ -82,5 +94,5 @@
         <child link="BR_uleg_link"/>
         <limit lower="-1.2217" upper="3.14" velocity="1" effort="7"/>
-        <dynamics friction="10.0"/>
+        <dynamics damping="0.01" friction="0.2"/>
     </joint>
     <!-- *********  BR_lleg  ********* -->
@@ -91,6 +103,12 @@
         <axis xyz="0 1 0"/>
         <limit lower="-1.57" upper="2.618" velocity="1" effort="7"/>
-        <xacro:lleg_jointDynamics></xacro:lleg_jointDynamics>
+        <dynamics damping="0.01" friction="0.2"/>
     </joint>
+     <!-- *********  BR_FOOT  ********* -->
+     <joint name="BR_foot_fixed" type="fixed">
+        <origin rpy="0 0 0" xyz="0.14 0 0"/>
+        <parent link="BR_lleg_link"/>
+        <child link="BR_foot"/>
+      </joint>
     <!-- *********  BL_hip  ********* -->
     <joint name="BL_hip_joint" type="revolute">
@@ -100,5 +118,5 @@
         <child link="BL_hip_link"/>
         <limit lower="-1.57" upper="1.57" velocity="1" effort="7"/>
-        <dynamics friction="10.0"/>
+        <dynamics damping="0.01" friction="0.2"/>
     </joint>
     <!-- *********  BL_uleg  ********* -->
@@ -109,5 +127,5 @@
         <child link="BL_uleg_link"/>
         <limit lower="-1.2217" upper="3.14" velocity="1" effort="7"/>
-        <dynamics friction="10.0"/>
+        <dynamics damping="0.01" friction="0.2"/>
     </joint>
     <!-- *********  BL_lleg  ********* -->
@@ -118,5 +136,11 @@
         <child link="BL_lleg_link"/>
         <limit lower="-1.57" upper="2.618" velocity="1" effort="7"/>
-        <xacro:lleg_jointDynamics></xacro:lleg_jointDynamics>
+        <dynamics damping="0.01" friction="0.2"/>
     </joint>
+    <!-- *********  BL_FOOT  ********* -->
+    <joint name="BL_foot_fixed" type="fixed">
+        <origin rpy="0 0 0" xyz="0.14 0 0"/>
+        <parent link="BL_lleg_link"/>
+        <child link="BL_foot"/>
+      </joint>
 </robot>

File: hyperdog_gazebo_sim/description/hyperdog_urdf_links.xacro (robot description, xacro)
@@ -108,4 +108,24 @@
         <xacro:inertial_right_lleg></xacro:inertial_right_lleg>
     </link>
+    <!-- *********** FR FOOT ********** -->
+    <link name="FR_foot">
+        <visual>
+          <origin rpy="0 0 0" xyz="0 0 0"/>
+          <geometry>
+            <sphere radius="0.02"/>
+          </geometry>
+          <material name="orange"/>
+        </visual>
+        <collision>
+          <origin rpy="0 0 0" xyz="0 0 0"/>
+          <geometry>
+            <sphere radius="0.03"/>
+          </geometry>
+        </collision>
+        <inertial>
+          <mass value="0.06"/>
+          <inertia ixx="9.6e-06" ixy="0.0" ixz="0.0" iyy="9.6e-06" iyz="0.0" izz="9.6e-06"/>
+        </inertial>
+      </link>
     <!-- *********** FL_hip ********** -->
     <link name="FL_hip_link">
@@ -165,4 +185,24 @@
         <xacro:inertial_left_lleg></xacro:inertial_left_lleg>
     </link>
+    <!-- *********** FL FOOT ********** -->
+    <link name="FL_foot">
+        <visual>
+          <origin rpy="0 0 0" xyz="0 0 0"/>
+          <geometry>
+            <sphere radius="0.02"/>
+          </geometry>
+          <material name="orange"/>
+        </visual>
+        <collision>
+          <origin rpy="0 0 0" xyz="0 0 0"/>
+          <geometry>
+            <sphere radius="0.03"/>
+          </geometry>
+        </collision>
+        <inertial>
+          <mass value="0.06"/>
+          <inertia ixx="9.6e-06" ixy="0.0" ixz="0.0" iyy="9.6e-06" iyz="0.0" izz="9.6e-06"/>
+        </inertial>
+      </link>
     <!-- *********** BR_hip ********** -->
     <link name="BR_hip_link">
@@ -222,4 +262,24 @@
         <xacro:inertial_right_lleg></xacro:inertial_right_lleg>
     </link>
+    <!-- *********** BR FOOT ********** -->
+    <link name="BR_foot">
+        <visual>
+          <origin rpy="0 0 0" xyz="0 0 0"/>
+          <geometry>
+            <sphere radius="0.02"/>
+          </geometry>
+          <material name="orange"/>
+        </visual>
+        <collision>
+          <origin rpy="0 0 0" xyz="0 0 0"/>
+          <geometry>
+            <sphere radius="0.03"/>
+          </geometry>
+        </collision>
+        <inertial>
+          <mass value="0.06"/>
+          <inertia ixx="9.6e-06" ixy="0.0" ixz="0.0" iyy="9.6e-06" iyz="0.0" izz="9.6e-06"/>
+        </inertial>
+      </link>
     <!-- *********** BL_hip ********** -->
     <link name="BL_hip_link">
@@ -279,3 +339,23 @@
         <xacro:inertial_left_lleg></xacro:inertial_left_lleg>
     </link>
+    <!-- *********** BL FOOT ********** -->
+    <link name="BL_foot">
+        <visual>
+          <origin rpy="0 0 0" xyz="0 0 0"/>
+          <geometry>
+            <sphere radius="0.02"/>
+          </geometry>
+          <material name="orange"/>
+        </visual>
+        <collision>
+          <origin rpy="0 0 0" xyz="0 0 0"/>
+          <geometry>
+            <sphere radius="0.03"/>
+          </geometry>
+        </collision>
+        <inertial>
+          <mass value="0.06"/>
+          <inertia ixx="9.6e-06" ixy="0.0" ixz="0.0" iyy="9.6e-06" iyz="0.0" izz="9.6e-06"/>
+        </inertial>
+      </link>
 </robot>

File: hyperdog_gazebo_sim/description/physics.xacro (robot description, xacro)
@@ -62,8 +62,10 @@
     <!-- Configure foot surface -->
     <xacro:macro name="foot_surface">
-        <mu1>1</mu1>
-        <mu2>1</mu2>
-        <minDepth>0.001</minDepth>
-        <fdir1>1 1 0</fdir1>
+        <mu1>0.2</mu1>
+        <mu2>0.2</mu2>
+        <self_collide>1</self_collide>
+        <material>Gazebo/DarkGrey</material>
+        <kp value="1000000.0"/>
+        <kd value="1.0"/>
     </xacro:macro>
 </robot>
