Commit message: updated urdf

File: hyperdog_gazebo_sim/description/hyperdog_gazebo.xacro (robot description, xacro)
@@ -11,118 +11,113 @@
 -->
     <xacro:include filename="physics.xacro" />
-    <gazebo reference="base_link">
-        <material>Gazebo/DarkGrey  </material>
+    <xacro:macro name="gz_hip">
         <mu1>0.2</mu1>
         <mu2>0.2</mu2>
-        <kp value="1000000.0"/>
-        <kd value="1.0"/>
-    </gazebo>
-    <gazebo reference="FR_hip_link">
+        <!-- <kp value="1000000.0"/>
+        <kd value="1.0"/> -->
+        <!-- <maxVel>0.0</maxVel> -->
+        <material>Gazebo/PioneerBody</material>
+    </xacro:macro>
+    <xacro:macro name="gz_uleg">
         <mu1>0.2</mu1>
         <mu2>0.2</mu2>
-        <material>Gazebo/PioneerBody</material>
+        <!-- <kp value="2147483647.0"/>
+        <kd value="1.0"/> -->
+        <!-- <maxVel>0.0</maxVel> -->
+        <!-- <self_collide>1</self_collide> -->
+        <material>Gazebo/Orange</material>
+    </xacro:macro>
+    <xacro:macro name="gz_lleg">
+        <mu1>0.2</mu1>
+        <mu2>0.2</mu2>
+        <!-- <kp>1000000.0</kp>
+        <kd>1.0</kd> -->
+        <!-- <maxVel>0.0</maxVel> -->
+        <!-- <self_collide>1</self_collide>  -->
+        <material>Gazebo/DarkYellow</material>
+    </xacro:macro>
+    <xacro:macro name="gz_foot">
+        <mu1>1.0</mu1>
+        <mu2>1.0</mu2>
+        <kp value="1000000.0" />
+        <kd value="100.0" />
+        <!-- <maxVel>0.0</maxVel> -->
+        <!-- <self_collide>1</self_collide> -->
+        <minDepth>0.001</minDepth>
+        <!-- <surface>
+            <friction>
+                <torsional>
+                    <coefficient>10</coefficient>
+                    <use_fatch_radius>false</use_fatch_radius>
+                    <surface_radius>0.1</surface_radius>
+                    <patch_radius>0.2</patch_radius>
+                </torsional>
+            </friction>
+            <contact>
+                <poissons_ratio>0.5</poissons_ratio>
+                <elastic_modulus>1e8</elastic_modulus>
+            </contact>
+        </surface> -->
+        <material>Gazebo/DarkGrey</material>
+    </xacro:macro>
+    <!-- body -->
+    <gazebo reference="base_link">
+        <mu1>0.05</mu1>
+        <mu2>0.05</mu2>
+        <!-- <kp>1000000.0</kp>
+        <kd>1.0</kd> -->
+        <material>Gazebo/DarkGrey  </material>
+    </gazebo>
+    <!-- hip -->
+    <gazebo reference="FR_hip_link">
+        <xacro:gz_hip></xacro:gz_hip>
     </gazebo>
     <gazebo reference="FL_hip_link">
-        <mu1>0.2</mu1>
-        <mu2>0.2</mu2>
-        <material>Gazebo/PioneerBody</material>
+        <xacro:gz_hip></xacro:gz_hip>
     </gazebo>
     <gazebo reference="BR_hip_link">
-        <mu1>0.2</mu1>
-        <mu2>0.2</mu2>
-        <material>Gazebo/PioneerBody</material>
+        <xacro:gz_hip></xacro:gz_hip>
     </gazebo>
     <gazebo reference="BL_hip_link">
-        <mu1>0.2</mu1>
-        <mu2>0.2</mu2>
-        <material>Gazebo/PioneerBody</material>
+        <xacro:gz_hip></xacro:gz_hip>
     </gazebo>
+    <!-- uleg -->
     <gazebo reference="FR_uleg_link">
-        <mu1>0.2</mu1>
-        <mu2>0.2</mu2>
-        <self_collide>1</self_collide>
-        <kp value="1000000.0"/>
-        <kd value="1.0"/>
-        <material>Gazebo/Orange</material>
+        <xacro:gz_uleg></xacro:gz_uleg>
     </gazebo>
     <gazebo reference="FL_uleg_link">
-        <mu1>0.2</mu1>
-        <mu2>0.2</mu2>
-        <self_collide>1</self_collide>
-        <kp value="1000000.0"/>
-        <kd value="1.0"/>
-        <material>Gazebo/Orange   </material>
+        <xacro:gz_uleg></xacro:gz_uleg>
     </gazebo>
     <gazebo reference="BR_uleg_link">
-        <mu1>0.2</mu1>
-        <mu2>0.2</mu2>
-        <self_collide>1</self_collide>
-        <kp value="1000000.0"/>
-        <kd value="1.0"/>
-        <material>Gazebo/Orange   </material>
+        <xacro:gz_uleg></xacro:gz_uleg>
     </gazebo>
     <gazebo reference="BL_uleg_link">
-        <mu1>0.2</mu1>
-        <mu2>0.2</mu2>
-        <self_collide>1</self_collide>
-        <kp value="1000000.0"/>
-        <kd value="1.0"/>
-        <material>Gazebo/Orange </material>
+        <xacro:gz_uleg></xacro:gz_uleg>
     </gazebo>
+    <!-- lleg -->
     <gazebo reference="FR_lleg_link">
-        <material>Gazebo/DarkYellow</material>
-        <mu1>0.2</mu1>
-        <mu2>0.2</mu2>
-        <self_collide>1</self_collide>
+        <xacro:gz_lleg></xacro:gz_lleg>
     </gazebo>
     <gazebo reference="FL_lleg_link">
-        <material>Gazebo/DarkYellow</material>
-        <mu1>0.2</mu1>
-        <mu2>0.2</mu2>
-        <self_collide>1</self_collide>
+        <xacro:gz_lleg></xacro:gz_lleg>
     </gazebo>
     <gazebo reference="BR_lleg_link">
-        <material>Gazebo/DarkYellow</material>
-        <mu1>0.2</mu1>
-        <mu2>0.2</mu2>
-        <self_collide>1</self_collide>
+        <xacro:gz_lleg></xacro:gz_lleg>
     </gazebo>
     <gazebo reference="BL_lleg_link">
-        <material>Gazebo/DarkYellow</material>
-        <mu1>0.2</mu1>
-        <mu2>0.2</mu2>
-        <self_collide>1</self_collide>
+        <xacro:gz_lleg></xacro:gz_lleg>
     </gazebo>
+    <!-- feet -->
     <gazebo reference="FR_foot">
-        <material>Gazebo/DarkGrey</material>
-        <mu1>0.6</mu1>
-        <mu2>0.6</mu2>
-        <self_collide>1</self_collide>
-        <kp value="1000000.0"/>
-        <kd value="1.0"/>
+        <xacro:gz_foot></xacro:gz_foot>
     </gazebo>
     <gazebo reference="FL_foot">
-        <material>Gazebo/DarkGrey</material>
-        <mu1>0.6</mu1>
-        <mu2>0.6</mu2>
-        <self_collide>1</self_collide>
-        <kp value="1000000.0"/>
-        <kd value="1.0"/>
+        <xacro:gz_foot></xacro:gz_foot>
     </gazebo>
     <gazebo reference="BL_foot">
-        <material>Gazebo/DarkGrey</material>
-        <mu1>0.6</mu1>
-        <mu2>0.6</mu2>
-        <self_collide>1</self_collide>
-        <kp value="1000000.0"/>
-        <kd value="1.0"/>
+        <xacro:gz_foot></xacro:gz_foot>
     </gazebo>
     <gazebo reference="BR_foot">
-        <material>Gazebo/DarkGrey</material>
-        <mu1>0.6</mu1>
-        <mu2>0.6</mu2>
-        <self_collide>1</self_collide>
-        <kp value="1000000.0"/>
-        <kd value="1.0"/>
+        <xacro:gz_foot></xacro:gz_foot>
     </gazebo>
 </robot>

File: hyperdog_gazebo_sim/description/hyperdog_urdf_joints.xacro (robot description, xacro)
@@ -7,10 +7,31 @@
                     <xacro:include filename="hyperdog_urdf_joints.xacro" />
     _____________________________________________________________________ -->
-    <!-- ******** Inertial ********** -->
+    <!-- joint dynamics -->
+    <xacro:property name="use_dynamics" value="true"/>
+    <xacro:macro name="hip_joint_dynamics">
+        <dynamics damping="1.0" friction="1.0"/>
+    </xacro:macro>
+    <xacro:macro name="uleg_joint_dynamics">
+        <dynamics damping="1.0" friction="1.0"/>
+    </xacro:macro>
+    <xacro:macro name="lleg_joint_dynamics">
+        <dynamics damping="1.0" friction="10.0"/>
+    </xacro:macro>
+    <!-- Limits -->
+    <xacro:macro name="hip_limits">
+        <limit lower="-1.57" upper="1.57" velocity="1" effort="27"/> <!-- effort = 7 -->
+    </xacro:macro>
+    <xacro:macro name="uleg_limits">
+        <limit lower="-1.2217" upper="3.14" velocity="1" effort="27"/>
+    </xacro:macro>
+    <xacro:macro name="lleg_limits">
+        <limit lower="-1.57" upper="2.618" velocity="1" effort="27"/>
+    </xacro:macro>
+    <!-- ******** Inertial - base joint ********** -->
     <joint name="inertial_joint" type="fixed">
         <parent link="base_link"/>
         <child link="inertial_link"/>
     </joint>
-    <!-- *********  FR_hip  ********* -->
+    <!-- *********  FR_hip joint ********* -->
     <joint name="FR_hip_joint" type="revolute">
         <axis xyz="-1 0 0"/>
@@ -18,8 +39,10 @@
         <parent link="base_link"/>
         <child link="FR_hip_link"/>
-        <limit lower="-1.57" upper="1.57" velocity="21" effort="7"/>
-        <dynamics damping="0.01" friction="0.2"/>
+        <xacro:hip_limits></xacro:hip_limits>
+        <xacro:if value="${use_dynamics}">
+            <xacro:hip_joint_dynamics></xacro:hip_joint_dynamics>
+        </xacro:if>
     </joint>
-    <!-- *********  FR_uleg  ********* -->
+    <!-- *********  FR_uleg joint ********* -->
     <joint name="FR_uleg_joint" type="revolute">
         <axis xyz="0 -1 0"/>
@@ -27,6 +50,8 @@
         <parent link="FR_hip_link"/>
         <child link="FR_uleg_link"/>
-        <limit lower="-1.2217" upper="3.14" velocity="1" effort="7"/>
-        <dynamics damping="0.01" friction="0.2"/>
+        <xacro:uleg_limits></xacro:uleg_limits>
+        <xacro:if value="${use_dynamics}">
+            <xacro:uleg_joint_dynamics></xacro:uleg_joint_dynamics>
+        </xacro:if>
     </joint>
     <!-- *********  FR_lleg  ********* -->
@@ -36,6 +61,8 @@
         <parent link="FR_uleg_link"/>
         <child link="FR_lleg_link"/>
-        <limit lower="-1.57" upper="2.618" velocity="1" effort="7"/>
-        <dynamics damping="0.01" friction="0.2"/>
+        <xacro:lleg_limits></xacro:lleg_limits>
+        <xacro:if value="${use_dynamics}">
+            <xacro:lleg_joint_dynamics></xacro:lleg_joint_dynamics>
+        </xacro:if>
     </joint>
      <!-- *********  FR_FOOT  ********* -->
@@ -51,6 +78,8 @@
         <parent link="base_link"/>
         <child link="FL_hip_link"/>
-        <limit lower="-1.57" upper="1.57" velocity="1" effort="7"/>
-        <dynamics damping="0.01" friction="0.2"/>
+        <xacro:hip_limits></xacro:hip_limits>
+        <xacro:if value="${use_dynamics}">
+            <xacro:hip_joint_dynamics></xacro:hip_joint_dynamics>
+        </xacro:if>
     </joint>
     <!-- *********  FL_uleg  ********* -->
@@ -60,6 +89,8 @@
         <parent link="FL_hip_link"/>
         <child link="FL_uleg_link"/>
-        <limit lower="-1.2217" upper="3.14" velocity="1" effort="7"/>
-        <dynamics damping="0.01" friction="0.2"/>
+        <xacro:uleg_limits></xacro:uleg_limits>
+        <xacro:if value="${use_dynamics}">
+            <xacro:uleg_joint_dynamics></xacro:uleg_joint_dynamics>
+        </xacro:if>
     </joint>
     <!-- *********  FL_lleg  ********* -->
@@ -69,6 +100,8 @@
         <parent link="FL_uleg_link"/>
         <child link="FL_lleg_link"/>
-        <limit lower="-1.57" upper="2.618" velocity="1" effort="7"/>
-        <dynamics damping="0.01" friction="0.2"/>
+        <xacro:lleg_limits></xacro:lleg_limits>
+        <xacro:if value="${use_dynamics}">
+            <xacro:lleg_joint_dynamics></xacro:lleg_joint_dynamics>
+        </xacro:if>
     </joint>
      <!-- *********  FL_FOOT  ********* -->
@@ -84,6 +117,8 @@
         <parent link="base_link"/>
         <child link="BR_hip_link"/>
-        <limit lower="-1.57" upper="1.57" velocity="1" effort="7"/>
-        <dynamics damping="0.01" friction="0.2"/>
+        <xacro:hip_limits></xacro:hip_limits>
+        <xacro:if value="${use_dynamics}">
+            <xacro:hip_joint_dynamics></xacro:hip_joint_dynamics>
+        </xacro:if>
     </joint>
     <!-- *********  BR_uleg  ********* -->
@@ -93,6 +128,8 @@
         <parent link="BR_hip_link"/>
         <child link="BR_uleg_link"/>
-        <limit lower="-1.2217" upper="3.14" velocity="1" effort="7"/>
-        <dynamics damping="0.01" friction="0.2"/>
+        <xacro:uleg_limits></xacro:uleg_limits>
+        <xacro:if value="${use_dynamics}">
+            <xacro:uleg_joint_dynamics></xacro:uleg_joint_dynamics>
+        </xacro:if>
     </joint>
     <!-- *********  BR_lleg  ********* -->
@@ -102,6 +139,8 @@
         <child link="BR_lleg_link"/>
         <axis xyz="0 1 0"/>
-        <limit lower="-1.57" upper="2.618" velocity="1" effort="7"/>
-        <dynamics damping="0.01" friction="0.2"/>
+        <xacro:lleg_limits></xacro:lleg_limits>
+        <xacro:if value="${use_dynamics}">
+            <xacro:lleg_joint_dynamics></xacro:lleg_joint_dynamics>
+        </xacro:if>
     </joint>
      <!-- *********  BR_FOOT  ********* -->
@@ -117,6 +156,8 @@
         <parent link="base_link"/>
         <child link="BL_hip_link"/>
-        <limit lower="-1.57" upper="1.57" velocity="1" effort="7"/>
-        <dynamics damping="0.01" friction="0.2"/>
+        <xacro:hip_limits></xacro:hip_limits>
+        <xacro:if value="${use_dynamics}">
+            <xacro:hip_joint_dynamics></xacro:hip_joint_dynamics>
+        </xacro:if>
     </joint>
     <!-- *********  BL_uleg  ********* -->
@@ -126,6 +167,8 @@
         <parent link="BL_hip_link"/>
         <child link="BL_uleg_link"/>
-        <limit lower="-1.2217" upper="3.14" velocity="1" effort="7"/>
-        <dynamics damping="0.01" friction="0.2"/>
+        <xacro:uleg_limits></xacro:uleg_limits>
+        <xacro:if value="${use_dynamics}">
+            <xacro:uleg_joint_dynamics></xacro:uleg_joint_dynamics>
+        </xacro:if>
     </joint>
     <!-- *********  BL_lleg  ********* -->
@@ -135,6 +178,8 @@
         <parent link="BL_uleg_link"/>
         <child link="BL_lleg_link"/>
-        <limit lower="-1.57" upper="2.618" velocity="1" effort="7"/>
-        <dynamics damping="0.01" friction="0.2"/>
+        <xacro:lleg_limits></xacro:lleg_limits>
+        <xacro:if value="${use_dynamics}">
+            <xacro:lleg_joint_dynamics></xacro:lleg_joint_dynamics>
+        </xacro:if>
     </joint>
     <!-- *********  BL_FOOT  ********* -->

File: hyperdog_gazebo_sim/description/hyperdog_urdf_links.xacro (robot description, xacro)
@@ -120,11 +120,8 @@
           <origin rpy="0 0 0" xyz="0 0 0"/>
           <geometry>
-            <sphere radius="0.03"/>
-          </geometry>
-        </collision>
-        <inertial>
-          <mass value="0.06"/>
-          <inertia ixx="9.6e-06" ixy="0.0" ixz="0.0" iyy="9.6e-06" iyz="0.0" izz="9.6e-06"/>
-        </inertial>
+            <sphere radius="0.021"/>
+          </geometry>
+        </collision>
+        <xacro:inertial_foot></xacro:inertial_foot>
       </link>
     <!-- *********** FL_hip ********** -->
@@ -197,11 +194,8 @@
           <origin rpy="0 0 0" xyz="0 0 0"/>
           <geometry>
-            <sphere radius="0.03"/>
-          </geometry>
-        </collision>
-        <inertial>
-          <mass value="0.06"/>
-          <inertia ixx="9.6e-06" ixy="0.0" ixz="0.0" iyy="9.6e-06" iyz="0.0" izz="9.6e-06"/>
-        </inertial>
+            <sphere radius="0.021"/>
+          </geometry>
+        </collision>
+        <xacro:inertial_foot></xacro:inertial_foot>
       </link>
     <!-- *********** BR_hip ********** -->
@@ -274,11 +268,8 @@
           <origin rpy="0 0 0" xyz="0 0 0"/>
           <geometry>
-            <sphere radius="0.03"/>
-          </geometry>
-        </collision>
-        <inertial>
-          <mass value="0.06"/>
-          <inertia ixx="9.6e-06" ixy="0.0" ixz="0.0" iyy="9.6e-06" iyz="0.0" izz="9.6e-06"/>
-        </inertial>
+            <sphere radius="0.021"/>
+          </geometry>
+        </collision>
+        <xacro:inertial_foot></xacro:inertial_foot>
       </link>
     <!-- *********** BL_hip ********** -->
@@ -351,11 +342,8 @@
           <origin rpy="0 0 0" xyz="0 0 0"/>
           <geometry>
-            <sphere radius="0.03"/>
-          </geometry>
-        </collision>
-        <inertial>
-          <mass value="0.06"/>
-          <inertia ixx="9.6e-06" ixy="0.0" ixz="0.0" iyy="9.6e-06" iyz="0.0" izz="9.6e-06"/>
-        </inertial>
+            <sphere radius="0.02"/>
+          </geometry>
+        </collision>
+        <xacro:inertial_foot></xacro:inertial_foot>
       </link>
 </robot>
