Commit message: updated urdf

File: hyperdog_gazebo_sim/description/physics.xacro (robot description, xacro)
@@ -2,10 +2,32 @@
 <robot xmlns:xacro="http://www.ros.org/wiki/xacro" >
     <!-- configure inertia -->
+    <xacro:property name="body_mass" value="4"/>
+    <xacro:property name="body_x_len" value="0.28"/>
+    <xacro:property name="body_y_len" value="0.172"/>
+    <xacro:property name="body_z_len" value="0.04"/>
+    <xacro:property name="hip_mass" value="0.3"/>
+    <xacro:property name="hip_x_len" value="0.05"/>
+    <xacro:property name="hip_y_len" value="0.03"/>
+    <xacro:property name="hip_z_len" value="0.04"/>
+    <xacro:property name="uleg_mass" value="0.5"/>
+    <xacro:property name="uleg_x_len" value="0.1"/>
+    <xacro:property name="uleg_y_len" value="0.02"/>
+    <xacro:property name="uleg_z_len" value="0.02"/>
+    <xacro:property name="lleg_mass" value="0.3"/>
+    <xacro:property name="lleg_x_len" value="0.1"/>
+    <xacro:property name="lleg_y_len" value="0.01"/>
+    <xacro:property name="lleg_z_len" value="0.01"/>
     <!--  BODY -->
     <xacro:macro name="inertial_body">
         <inertial>
             <origin xyz="-0.006 0.00633 0.00214" rpy="0 0 0"/> <!-- 0.006, -0.000233, 0.00214 -->
-            <mass value="2.0" />
-            <inertia ixx="0.00728" ixy="0.00003" ixz="0.00073" iyy="0.01641" iyz="0.00013" izz="0.01965" />
+            <mass value="${body_mass}" />
+            <inertia ixx="${(1/12) * body_mass * (body_y_len * body_y_len + body_z_len * body_z_len)}" ixy="0.0" ixz="0.0"
+                     iyy="${(1/12) * body_mass * (body_x_len * body_x_len + body_z_len * body_z_len)}" iyz="0.0"
+                     izz="${(1/12) * body_mass * (body_x_len * body_x_len + body_y_len * body_y_len)}" />
+            <!-- <mass value="2.0"/>
+            <inertia ixx="0.00728" ixy="0.00003" ixz="0.00073"
+                     iyy="0.01641" iyz="0.00013" izz="0.01965"/>
+             -->
         </inertial>
     </xacro:macro>
@@ -14,6 +36,11 @@
         <inertial>
             <origin xyz="0.0 -0.02 0.01" rpy="0 0 0"/>
-            <mass value="0.25" />
-            <inertia ixx="0.00199" ixy="0.00339" ixz="0.00075" iyy="0.0078" iyz="0.00034" izz="0.00943" />
+            <mass value="${hip_mass}" />
+            <inertia ixx="${(1/12) * hip_mass * (hip_y_len * hip_y_len + hip_z_len * hip_z_len)}" ixy="0.0" ixz="0.0"
+                     iyy="${(1/12) * hip_mass * (hip_x_len * hip_x_len + hip_z_len * hip_z_len)}" iyz="0.0"
+                     izz="${(1/12) * hip_mass * (hip_x_len * hip_x_len + hip_y_len * hip_y_len)}" />
+            <!-- <mass value="0.25"/>
+            <inertia ixx="0.00199" ixy="0.00339" ixz="0.00075"
+                    iyy="0.0078" iyz="0.00034" izz="0.00943"/> -->
         </inertial>
     </xacro:macro>
@@ -21,6 +48,11 @@
         <inertial>
             <origin xyz="0.0 0.02 0.01" rpy="0 0 0"/>
-            <mass value="0.25" />
-            <inertia ixx="0.00199" ixy="0.00339" ixz="0.00075" iyy="0.0078" iyz="0.00034" izz="0.00943" />
+            <mass value="${hip_mass}" />
+            <inertia ixx="${(1/12) * hip_mass * (hip_y_len * hip_y_len + hip_z_len * hip_z_len)}" ixy="0.0" ixz="0.0"
+                     iyy="${(1/12) * hip_mass * (hip_x_len * hip_x_len + hip_z_len * hip_z_len)}" iyz="0.0"
+                     izz="${(1/12) * hip_mass * (hip_x_len * hip_x_len + hip_y_len * hip_y_len)}" />
+            <!-- <mass value="0.25"/>
+            <inertia ixx="0.00199" ixy="0.00339" ixz="0.00075"
+                     iyy="0.0078" iyz="0.00034" izz="0.00943"/> -->
         </inertial>
     </xacro:macro>
@@ -29,6 +61,11 @@
         <inertial>
             <origin xyz="-0.02 0.02 0.0" rpy="0 0 0"/>
-            <mass value="0.35" />
-            <inertia ixx="0.007467" ixy="0.009383" ixz="0.000515" iyy="0.012791" iyz="0.000298" izz="0.019903" />
+            <!-- <mass value="${uleg_mass}" />
+            <inertia ixx="${(1/12) * uleg_mass * (uleg_y_len * uleg_y_len + uleg_z_len * uleg_z_len)}" ixy="0.0" ixz="0.0"
+                     iyy="${(1/12) * uleg_mass * (uleg_x_len * uleg_x_len + uleg_z_len * uleg_z_len)}" iyz="0.0"
+                     izz="${(1/12) * uleg_mass * (uleg_x_len * uleg_x_len + uleg_y_len * uleg_y_len)}" /> -->
+            <mass value="0.35"/>
+            <inertia ixx="0.007467" ixy="0.009383" ixz="0.000515"
+                     iyy="0.012791" iyz="0.000298" izz="0.019903"/>
         </inertial>
     </xacro:macro>
@@ -36,6 +73,11 @@
         <inertial>
             <origin xyz="-0.02 -0.02 0.0" rpy="0 0 0"/>
-            <mass value="0.35" />
-            <inertia ixx="0.007467" ixy="0.009383" ixz="0.000515" iyy="0.012791" iyz="0.000298" izz="0.019903" />
+            <!-- <mass value="${uleg_mass}"/>
+            <inertia ixx="${(1/12) * uleg_mass * (uleg_y_len * uleg_y_len + uleg_z_len * uleg_z_len)}" ixy="0.0" ixz="0.0"
+                     iyy="${(1/12) * uleg_mass * (uleg_x_len * uleg_x_len + uleg_z_len * uleg_z_len)}" iyz="0.0"
+                     izz="${(1/12) * uleg_mass * (uleg_x_len * uleg_x_len + uleg_y_len * uleg_y_len)}" /> -->
+            <mass value="0.35"/>
+            <inertia ixx="0.007467" ixy="0.009383" ixz="0.000515"
+                    iyy="0.012791" iyz="0.000298" izz="0.019903"/>
         </inertial>
     </xacro:macro>
@@ -44,6 +86,11 @@
         <inertial>
             <origin xyz="0.05 0.0 -0.0" rpy="0 0 0"/>
-            <mass value="0.24" />
-            <inertia ixx="0.01273" ixy="0.01054" ixz="0.00877" iyy="0.02196" iyz="0.00602" izz="0.02318" />
+            <!-- <mass value="${lleg_mass}" />
+            <inertia ixx="${(1/12) * lleg_mass * (lleg_y_len * lleg_y_len + lleg_z_len * lleg_z_len)}" ixy="0.0" ixz="0.0"
+                     iyy="${(1/12) * lleg_mass * (lleg_x_len * lleg_x_len + lleg_z_len * lleg_z_len)}" iyz="0.0"
+                     izz="${(1/12) * lleg_mass * (lleg_x_len * lleg_x_len + lleg_y_len * lleg_y_len)}" /> -->
+            <mass value="0.24"/>
+            <inertia ixx="0.01273" ixy="0.01054" ixz="0.00877"
+                    iyy="0.02196" iyz="0.00602" izz="0.02318"/>
         </inertial>
     </xacro:macro>
@@ -51,21 +98,19 @@
         <inertial>
             <origin xyz="0.05 0.0 -0.0" rpy="0 0 0"/>
-            <mass value="0.24" />
-            <inertia ixx="0.01273" ixy="0.01054" ixz="0.00877" iyy="0.02196" iyz="0.00602" izz="0.02318" />
+            <!-- <mass value="${lleg_mass}" />
+            <inertia ixx="${(1/12) * lleg_mass * (lleg_y_len * lleg_y_len + lleg_z_len * lleg_z_len)}" ixy="0.0" ixz="0.0"
+                     iyy="${(1/12) * lleg_mass * (lleg_x_len * lleg_x_len + lleg_z_len * lleg_z_len)}" iyz="0.0"
+                     izz="${(1/12) * lleg_mass * (lleg_x_len * lleg_x_len + lleg_y_len * lleg_y_len)}" /> -->
+            <mass value="0.24"/>
+            <inertia ixx="0.01273" ixy="0.01054" ixz="0.00877"
+                    iyy="0.02196" iyz="0.00602" izz="0.02318"/>
+        </inertial>
+    </xacro:macro>
+    <xacro:macro name="inertial_foot">
+        <inertial>
+            <mass value="0.06"/>
+            <inertia ixx="9.6e-06" ixy="0.0" ixz="0.0" iyy="9.6e-06" iyz="0.0" izz="9.6e-06"/>
         </inertial>
     </xacro:macro>
     <!-- ************************************************************************************************** -->
-    <!-- Configure joint dynamics -->
-    <xacro:macro name="lleg_jointDynamics">
-        <dynamics damping="1.0" friction="1000.0"/>
-    </xacro:macro>
-    <!-- Configure foot surface -->
-    <xacro:macro name="foot_surface">
-        <mu1>0.2</mu1>
-        <mu2>0.2</mu2>
-        <self_collide>1</self_collide>
-        <material>Gazebo/DarkGrey</material>
-        <kp value="1000000.0"/>
-        <kd value="1.0"/>
-    </xacro:macro>
 </robot>

Commit message: udated launch and urdf

File: hyperdog_gazebo_sim/description/hyperdog_gazebo.xacro (robot description, xacro)
@@ -27,4 +27,6 @@
         <!-- <self_collide>1</self_collide> -->
         <material>Gazebo/Orange</material>
+        <!-- <implicitSpringDamper>1</implicitSpringDamper>
+        <springStiffness>100</springStiffness> -->
     </xacro:macro>
     <xacro:macro name="gz_lleg">
@@ -36,4 +38,6 @@
         <!-- <self_collide>1</self_collide>  -->
         <material>Gazebo/DarkYellow</material>
+        <!-- <implicitSpringDamper>1</implicitSpringDamper>
+        <springStiffness>100</springStiffness> -->
     </xacro:macro>
     <xacro:macro name="gz_foot">
@@ -45,18 +49,4 @@
         <!-- <self_collide>1</self_collide> -->
         <minDepth>0.001</minDepth>
-        <!-- <surface>
-            <friction>
-                <torsional>
-                    <coefficient>10</coefficient>
-                    <use_fatch_radius>false</use_fatch_radius>
-                    <surface_radius>0.1</surface_radius>
-                    <patch_radius>0.2</patch_radius>
-                </torsional>
-            </friction>
-            <contact>
-                <poissons_ratio>0.5</poissons_ratio>
-                <elastic_modulus>1e8</elastic_modulus>
-            </contact>
-        </surface> -->
         <material>Gazebo/DarkGrey</material>
     </xacro:macro>

File: hyperdog_gazebo_sim/description/hyperdog_urdf_joints.xacro (robot description, xacro)
@@ -7,26 +7,16 @@
                     <xacro:include filename="hyperdog_urdf_joints.xacro" />
     _____________________________________________________________________ -->
-    <!-- joint dynamics -->
-    <xacro:property name="use_dynamics" value="true"/>
-    <xacro:macro name="hip_joint_dynamics">
-        <dynamics damping="1.0" friction="1.0"/>
-    </xacro:macro>
-    <xacro:macro name="uleg_joint_dynamics">
-        <dynamics damping="1.0" friction="1.0"/>
-    </xacro:macro>
-    <xacro:macro name="lleg_joint_dynamics">
-        <dynamics damping="1.0" friction="10.0"/>
-    </xacro:macro>
+    <xacro:include filename="consts.xacro" />
     <!-- Limits -->
     <xacro:macro name="hip_limits">
-        <limit lower="-1.57" upper="1.57" velocity="1" effort="27"/> <!-- effort = 7 -->
+        <limit lower="${hip_low_limit}" upper="${hip_up_limit}" velocity="${velocity}" effort="${effort}"/> <!-- effort = 7 -->
     </xacro:macro>
     <xacro:macro name="uleg_limits">
-        <limit lower="-1.2217" upper="3.14" velocity="1" effort="27"/>
+        <limit lower="${uleg_low_limit}" upper="${uleg_up_limit}" velocity="${velocity}" effort="${effort}"/>
     </xacro:macro>
     <xacro:macro name="lleg_limits">
-        <limit lower="-1.57" upper="2.618" velocity="1" effort="27"/>
+        <limit lower="${lleg_low_limit}" upper="${lleg_up_limit}" velocity="${velocity}" effort="${effort}"/>
     </xacro:macro>
-    <!-- ******** Inertial - base joint ********** -->
+    <!-- ******** Inertial-base joint ********** -->
     <joint name="inertial_joint" type="fixed">
         <parent link="base_link"/>
@@ -39,4 +29,37 @@
         <parent link="base_link"/>
         <child link="FR_hip_link"/>
+        <xacro:hip_limits></xacro:hip_limits>
+        <xacro:if value="${use_dynamics}">
+            <xacro:hip_joint_dynamics></xacro:hip_joint_dynamics>
+        </xacro:if>
+    </joint>
+    <!-- *********  FL_hip  ********* -->
+    <joint name="FL_hip_joint" type="revolute">
+        <axis xyz="1 0 0"/>
+        <origin xyz="0.175 0.066 0" rpy="0 0 0"/>
+        <parent link="base_link"/>
+        <child link="FL_hip_link"/>
+        <xacro:hip_limits></xacro:hip_limits>
+        <xacro:if value="${use_dynamics}">
+            <xacro:hip_joint_dynamics></xacro:hip_joint_dynamics>
+        </xacro:if>
+    </joint>
+    <!-- *********  BR_hip  ********* -->
+    <joint name="BR_hip_joint" type="revolute">
+        <axis xyz="-1 0 0"/>
+        <origin xyz="-0.175 -0.066 0" rpy="0 0 0"/>
+        <parent link="base_link"/>
+        <child link="BR_hip_link"/>
+        <xacro:hip_limits></xacro:hip_limits>
+        <xacro:if value="${use_dynamics}">
+            <xacro:hip_joint_dynamics></xacro:hip_joint_dynamics>
+        </xacro:if>
+    </joint>
+    <!-- *********  BL_hip  ********* -->
+    <joint name="BL_hip_joint" type="revolute">
+        <axis xyz="1 0 0"/>
+        <origin xyz="-0.175 0.066 0" rpy="0 0 0"/>
+        <parent link="base_link"/>
+        <child link="BL_hip_link"/>
         <xacro:hip_limits></xacro:hip_limits>
         <xacro:if value="${use_dynamics}">
@@ -55,4 +78,37 @@
         </xacro:if>
     </joint>
+    <!-- *********  FL_uleg  ********* -->
+    <joint name="FL_uleg_joint" type="revolute">
+        <axis xyz="0 -1 0"/>
+        <origin xyz="0 0.104 0" rpy="0 0 0"/>
+        <parent link="FL_hip_link"/>
+        <child link="FL_uleg_link"/>
+        <xacro:uleg_limits></xacro:uleg_limits>
+        <xacro:if value="${use_dynamics}">
+            <xacro:uleg_joint_dynamics></xacro:uleg_joint_dynamics>
+        </xacro:if>
+    </joint>
+    <!-- *********  BR_uleg  ********* -->
+    <joint name="BR_uleg_joint" type="revolute">
+        <axis xyz="0 -1 0"/>
+        <origin xyz="0 -0.104 0" rpy="0 0 0"/>
+        <parent link="BR_hip_link"/>
+        <child link="BR_uleg_link"/>
+        <xacro:uleg_limits></xacro:uleg_limits>
+        <xacro:if value="${use_dynamics}">
+            <xacro:uleg_joint_dynamics></xacro:uleg_joint_dynamics>
+        </xacro:if>
+    </joint>
+    <!-- *********  BL_uleg  ********* -->
+    <joint name="BL_uleg_joint" type="revolute">
+        <axis xyz="0 -1 0"/>
+        <origin xyz="0 0.104 0" rpy="0 0 0"/>
+        <parent link="BL_hip_link"/>
+        <child link="BL_uleg_link"/>
+        <xacro:uleg_limits></xacro:uleg_limits>
+        <xacro:if value="${use_dynamics}">
+            <xacro:uleg_joint_dynamics></xacro:uleg_joint_dynamics>
+        </xacro:if>
+    </joint>
     <!-- *********  FR_lleg  ********* -->
     <joint name="FR_lleg_joint" type="revolute">
@@ -64,32 +120,4 @@
         <xacro:if value="${use_dynamics}">
             <xacro:lleg_joint_dynamics></xacro:lleg_joint_dynamics>
-        </xacro:if>
-    </joint>
-     <!-- *********  FR_FOOT  ********* -->
-     <joint name="FR_foot_fixed" type="fixed">
-        <origin rpy="0 0 0" xyz="0.14 0 0"/>
-        <parent link="FR_lleg_link"/>
-        <child link="FR_foot"/>
-      </joint>
-    <!-- *********  FL_hip  ********* -->
-    <joint name="FL_hip_joint" type="revolute">
-        <axis xyz="1 0 0"/>
-        <origin xyz="0.175 0.066 0" rpy="0 0 0"/>
-        <parent link="base_link"/>
-        <child link="FL_hip_link"/>
-        <xacro:hip_limits></xacro:hip_limits>
-        <xacro:if value="${use_dynamics}">
-            <xacro:hip_joint_dynamics></xacro:hip_joint_dynamics>
-        </xacro:if>
-    </joint>
-    <!-- *********  FL_uleg  ********* -->
-    <joint name="FL_uleg_joint" type="revolute">
-        <axis xyz="0 -1 0"/>
-        <origin xyz="0 0.104 0" rpy="0 0 0"/>
-        <parent link="FL_hip_link"/>
-        <child link="FL_uleg_link"/>
-        <xacro:uleg_limits></xacro:uleg_limits>
-        <xacro:if value="${use_dynamics}">
-            <xacro:uleg_joint_dynamics></xacro:uleg_joint_dynamics>
         </xacro:if>
     </joint>
@@ -105,32 +133,4 @@
         </xacro:if>
     </joint>
-     <!-- *********  FL_FOOT  ********* -->
-     <joint name="FL_foot_fixed" type="fixed">
-        <origin rpy="0 0 0" xyz="0.14 0 0"/>
-        <parent link="FL_lleg_link"/>
-        <child link="FL_foot"/>
-      </joint>
-    <!-- *********  BR_hip  ********* -->
-    <joint name="BR_hip_joint" type="revolute">
-        <axis xyz="-1 0 0"/>
-        <origin xyz="-0.175 -0.066 0" rpy="0 0 0"/>
-        <parent link="base_link"/>
-        <child link="BR_hip_link"/>
-        <xacro:hip_limits></xacro:hip_limits>
-        <xacro:if value="${use_dynamics}">
-            <xacro:hip_joint_dynamics></xacro:hip_joint_dynamics>
-        </xacro:if>
-    </joint>
-    <!-- *********  BR_uleg  ********* -->
-    <joint name="BR_uleg_joint" type="revolute">
-        <axis xyz="0 -1 0"/>
-        <origin xyz="0 -0.104 0" rpy="0 0 0"/>
-        <parent link="BR_hip_link"/>
-        <child link="BR_uleg_link"/>
-        <xacro:uleg_limits></xacro:uleg_limits>
-        <xacro:if value="${use_dynamics}">
-            <xacro:uleg_joint_dynamics></xacro:uleg_joint_dynamics>
-        </xacro:if>
-    </joint>
     <!-- *********  BR_lleg  ********* -->
     <joint name="BR_lleg_joint" type="revolute">
@@ -142,32 +142,4 @@
         <xacro:if value="${use_dynamics}">
             <xacro:lleg_joint_dynamics></xacro:lleg_joint_dynamics>
-        </xacro:if>
-    </joint>
-     <!-- *********  BR_FOOT  ********* -->
-     <joint name="BR_foot_fixed" type="fixed">
-        <origin rpy="0 0 0" xyz="0.14 0 0"/>
-        <parent link="BR_lleg_link"/>
-        <child link="BR_foot"/>
-      </joint>
-    <!-- *********  BL_hip  ********* -->
-    <joint name="BL_hip_joint" type="revolute">
-        <axis xyz="1 0 0"/>
-        <origin xyz="-0.175 0.066 0" rpy="0 0 0"/>
-        <parent link="base_link"/>
-        <child link="BL_hip_link"/>
-        <xacro:hip_limits></xacro:hip_limits>
-        <xacro:if value="${use_dynamics}">
-            <xacro:hip_joint_dynamics></xacro:hip_joint_dynamics>
-        </xacro:if>
-    </joint>
-    <!-- *********  BL_uleg  ********* -->
-    <joint name="BL_uleg_joint" type="revolute">
-        <axis xyz="0 -1 0"/>
-        <origin xyz="0 0.104 0" rpy="0 0 0"/>
-        <parent link="BL_hip_link"/>
-        <child link="BL_uleg_link"/>
-        <xacro:uleg_limits></xacro:uleg_limits>
-        <xacro:if value="${use_dynamics}">
-            <xacro:uleg_joint_dynamics></xacro:uleg_joint_dynamics>
         </xacro:if>
     </joint>
@@ -183,4 +155,22 @@
         </xacro:if>
     </joint>
+     <!-- *********  FR_FOOT  ********* -->
+     <joint name="FR_foot_fixed" type="fixed">
+        <origin rpy="0 0 0" xyz="0.14 0 0"/>
+        <parent link="FR_lleg_link"/>
+        <child link="FR_foot"/>
+      </joint>
+     <!-- *********  FL_FOOT  ********* -->
+     <joint name="FL_foot_fixed" type="fixed">
+        <origin rpy="0 0 0" xyz="0.14 0 0"/>
+        <parent link="FL_lleg_link"/>
+        <child link="FL_foot"/>
+      </joint>
+     <!-- *********  BR_FOOT  ********* -->
+     <joint name="BR_foot_fixed" type="fixed">
+        <origin rpy="0 0 0" xyz="0.14 0 0"/>
+        <parent link="BR_lleg_link"/>
+        <child link="BR_foot"/>
+      </joint>
     <!-- *********  BL_FOOT  ********* -->
     <joint name="BL_foot_fixed" type="fixed">
