Commit message: udated launch and urdf

File: hyperdog_gazebo_sim/description/hyperdog_urdf_links.xacro (robot description, xacro)
@@ -9,4 +9,5 @@
                     <xacro:include filename="hyperdog_urdf_links.xacro" />
     _____________________________________________________________________ -->
+    <xacro:include filename="consts.xacro" />
     <xacro:include filename="physics.xacro" />
     <!-- load meshes -->
@@ -51,4 +52,5 @@
         </collision>
     </link>
+    <!-- !!!!!!!!!!!!!!!!!!!!!!! HIPS !!!!!!!!!!!!!!!!!!!!!!!!!!!! -->
     <!-- *********** FR_hip *********** -->
     <link name="FR_hip_link">
@@ -70,4 +72,62 @@
         <xacro:inertial_right_hip></xacro:inertial_right_hip>
     </link>
+    <!-- *********** FL_hip ********** -->
+    <link name="FL_hip_link">
+        <visual>
+            <origin xyz="0 0 0" rpy="0 0 0"/>
+            <geometry>
+                <xacro:leftHip_mesh></xacro:leftHip_mesh>
+            </geometry>
+            <material name="red">
+                <color rgba="0.8 0.2 0.2 1"/>
+            </material>
+        </visual>
+        <collision>
+            <origin xyz="0 0 0" rpy="0 0 0"/>
+            <geometry>
+                <xacro:leftHip_mesh></xacro:leftHip_mesh>
+            </geometry>
+        </collision>
+        <xacro:inertial_left_hip></xacro:inertial_left_hip>
+    </link>
+    <!-- *********** BR_hip ********** -->
+    <link name="BR_hip_link">
+        <visual>
+            <origin xyz="0 0 0" rpy="0 0 0"/>
+            <geometry>
+                <xacro:rightHip_mesh></xacro:rightHip_mesh>
+            </geometry>
+            <material name="red">
+                <color rgba="0.8 0.2 0.2 1"/>
+            </material>
+        </visual>
+        <collision>
+            <origin xyz="0 0 0" rpy="0 0 0"/>
+            <geometry>
+                <xacro:rightHip_mesh></xacro:rightHip_mesh>
+            </geometry>
+        </collision>
+        <xacro:inertial_right_hip></xacro:inertial_right_hip>
+    </link>
+    <!-- *********** BL_hip ********** -->
+    <link name="BL_hip_link">
+        <visual>
+            <origin xyz="0 0 0" rpy="0 0 0"/>
+            <geometry>
+                <xacro:leftHip_mesh></xacro:leftHip_mesh>
+            </geometry>
+            <material name="red">
+                <color rgba="0.8 0.2 0.2 1"/>
+            </material>
+        </visual>
+        <collision>
+            <origin xyz="0 0 0" rpy="0 0 0"/>
+            <geometry>
+                <xacro:leftHip_mesh></xacro:leftHip_mesh>
+            </geometry>
+        </collision>
+        <xacro:inertial_left_hip></xacro:inertial_left_hip>
+    </link>
+    <!-- !!!!!!!!!!!!!!!!!!!!!!! ULEGs !!!!!!!!!!!!!!!!!!!!!!!!!!!! -->
     <!-- *********** FR_uleg ********** -->
     <link name="FR_uleg_link">
@@ -89,4 +149,62 @@
         <xacro:inertial_right_uleg></xacro:inertial_right_uleg>
     </link>
+    <!-- *********** FL_uleg ********** -->
+    <link name="FL_uleg_link">
+        <visual>
+            <origin xyz="0 0 0" rpy="0 0 0"/>
+            <geometry>
+                <xacro:leftUleg_mesh></xacro:leftUleg_mesh>
+            </geometry>
+            <material name="orange">
+                <color rgba="0.8 0.5 0.8 1"/>
+            </material>
+        </visual>
+        <collision>
+            <origin xyz="0 0 0" rpy="0 0 0"/>
+            <geometry>
+                <xacro:leftUleg_mesh></xacro:leftUleg_mesh>
+            </geometry>
+        </collision>
+        <xacro:inertial_left_uleg></xacro:inertial_left_uleg>
+    </link>
+    <!-- *********** BR_uleg ********** -->
+    <link name="BR_uleg_link">
+        <visual>
+            <origin xyz="0 0 0" rpy="0 0 0"/>
+            <geometry>
+                <xacro:rightUleg_mesh></xacro:rightUleg_mesh>
+            </geometry>
+            <material name="orange">
+                <color rgba="0.8 0.5 0.8 1"/>
+            </material>
+        </visual>
+        <collision>
+            <origin xyz="0 0 0" rpy="0 0 0"/>
+            <geometry>
+                <xacro:rightUleg_mesh></xacro:rightUleg_mesh>
+            </geometry>
+        </collision>
+        <xacro:inertial_right_uleg></xacro:inertial_right_uleg>
+    </link>
+    <!-- *********** BL_uleg ********** -->
+    <link name="BL_uleg_link">
+        <visual>
+            <origin xyz="0 0 0" rpy="0 0 0"/>
+            <geometry>
+                <xacro:leftUleg_mesh></xacro:leftUleg_mesh>
+            </geometry>
+            <material name="orange">
+                <color rgba="0.8 0.5 0.8 1"/>
+            </material>
+        </visual>
+        <collision>
+            <origin xyz="0 0 0" rpy="0 0 0"/>
+            <geometry>
+                <xacro:leftUleg_mesh></xacro:leftUleg_mesh>
+            </geometry>
+        </collision>
+        <xacro:inertial_left_uleg></xacro:inertial_left_uleg>
+    </link>
+    <!-- !!!!!!!!!!!!!!!!!!!!!!! LLEGs !!!!!!!!!!!!!!!!!!!!!!!!!!!! -->
     <!-- *********** FR_lleg ********** -->
     <link name="FR_lleg_link">
@@ -108,4 +226,79 @@
         <xacro:inertial_right_lleg></xacro:inertial_right_lleg>
     </link>
+    <!-- *********** FL_lleg ********** -->
+    <link name="FL_lleg_link">
+        <visual>
+            <origin xyz="0 0 0" rpy="0 0 0"/>
+            <geometry>
+                <xacro:lleg_mesh></xacro:lleg_mesh>
+            </geometry>
+            <material name="yellow">
+                <color rgba="0.8 1.0 0.1 1"/>
+            </material>
+        </visual>
+        <collision>
+            <origin xyz="0 0 0" rpy="0 0 0"/>
+            <geometry>
+                <xacro:lleg_mesh></xacro:lleg_mesh>
+            </geometry>
+        </collision>
+        <xacro:inertial_left_lleg></xacro:inertial_left_lleg>
+    </link>
+      <!-- *********** BR_lleg ********** -->
+    <link name="BR_lleg_link">
+        <visual>
+            <origin xyz="0 0 0" rpy="0 0 0"/>
+            <geometry>
+                <xacro:lleg_mesh></xacro:lleg_mesh>
+            </geometry>
+            <material name="yellow">
+                <color rgba="0.8 1.0 0.1 1"/>
+            </material>
+        </visual>
+        <collision>
+            <origin xyz="0 0 0" rpy="0 0 0"/>
+            <geometry>
+                <xacro:lleg_mesh></xacro:lleg_mesh>
+            </geometry>
+        </collision>
+        <xacro:inertial_right_lleg></xacro:inertial_right_lleg>
+    </link>
+    <!-- *********** BL_lleg ********** -->
+    <link name="BL_lleg_link">
+        <visual>
+            <origin xyz="0 0 0" rpy="0 0 0"/>
+            <geometry>
+                <xacro:lleg_mesh></xacro:lleg_mesh>
+            </geometry>
+            <material name="yellow">
+                <color rgba="0.8 1.0 0.1 1"/>
+            </material>
+        </visual>
+        <collision>
+            <origin xyz="0 0 0" rpy="0 0 0"/>
+            <geometry>
+                <xacro:lleg_mesh></xacro:lleg_mesh>
+            </geometry>
+        </collision>
+        <xacro:inertial_left_lleg></xacro:inertial_left_lleg>
+    </link>
+    <!-- !!!!!!!!!!!!!!!!!!!!!!! FEET !!!!!!!!!!!!!!!!!!!!!!!!!!!! -->
+    <!-- *********** FL FOOT ********** -->
+    <link name="FL_foot">
+        <visual>
+          <origin rpy="0 0 0" xyz="0 0 0"/>
+          <geometry>
+            <sphere radius="${foot_radius}"/>
+          </geometry>
+          <material name="orange"/>
+        </visual>
+        <collision>
+          <origin rpy="0 0 0" xyz="0 0 0"/>
+          <geometry>
+            <sphere radius="${foot_radius}"/>
+          </geometry>
+        </collision>
+        <xacro:inertial_foot></xacro:inertial_foot>
+      </link>
     <!-- *********** FR FOOT ********** -->
     <link name="FR_foot">
@@ -113,5 +306,5 @@
           <origin rpy="0 0 0" xyz="0 0 0"/>
           <geometry>
-            <sphere radius="0.02"/>
+            <sphere radius="${foot_radius}"/>
           </geometry>
           <material name="orange"/>
@@ -120,72 +313,15 @@
           <origin rpy="0 0 0" xyz="0 0 0"/>
           <geometry>
-            <sphere radius="0.021"/>
+            <sphere radius="${foot_radius}"/>
           </geometry>
         </collision>
         <xacro:inertial_foot></xacro:inertial_foot>
       </link>
-    <!-- *********** FL_hip ********** -->
-    <link name="FL_hip_link">
-        <visual>
-            <origin xyz="0 0 0" rpy="0 0 0"/>
-            <geometry>
-                <xacro:leftHip_mesh></xacro:leftHip_mesh>
-            </geometry>
-            <material name="red">
-                <color rgba="0.8 0.2 0.2 1"/>
-            </material>
-        </visual>
-        <collision>
-            <origin xyz="0 0 0" rpy="0 0 0"/>
-            <geometry>
-                <xacro:leftHip_mesh></xacro:leftHip_mesh>
-            </geometry>
-        </collision>
-        <xacro:inertial_left_hip></xacro:inertial_left_hip>
-    </link>
-    <!-- *********** FL_uleg ********** -->
-    <link name="FL_uleg_link">
-        <visual>
-            <origin xyz="0 0 0" rpy="0 0 0"/>
-            <geometry>
-                <xacro:leftUleg_mesh></xacro:leftUleg_mesh>
-            </geometry>
-            <material name="orange">
-                <color rgba="0.8 0.5 0.8 1"/>
-            </material>
-        </visual>
-        <collision>
-            <origin xyz="0 0 0" rpy="0 0 0"/>
-            <geometry>
-                <xacro:leftUleg_mesh></xacro:leftUleg_mesh>
-            </geometry>
-        </collision>
-        <xacro:inertial_left_uleg></xacro:inertial_left_uleg>
-    </link>
-    <!-- *********** FL_lleg ********** -->
-    <link name="FL_lleg_link">
-        <visual>
-            <origin xyz="0 0 0" rpy="0 0 0"/>
-            <geometry>
-                <xacro:lleg_mesh></xacro:lleg_mesh>
-            </geometry>
-            <material name="yellow">
-                <color rgba="0.8 1.0 0.1 1"/>
-            </material>
-        </visual>
-        <collision>
-            <origin xyz="0 0 0" rpy="0 0 0"/>
-            <geometry>
-                <xacro:lleg_mesh></xacro:lleg_mesh>
-            </geometry>
-        </collision>
-        <xacro:inertial_left_lleg></xacro:inertial_left_lleg>
-    </link>
-    <!-- *********** FL FOOT ********** -->
-    <link name="FL_foot">
-        <visual>
-          <origin rpy="0 0 0" xyz="0 0 0"/>
-          <geometry>
-            <sphere radius="0.02"/>
+    <!-- *********** BR FOOT ********** -->
+    <link name="BR_foot">
+        <visual>
+          <origin rpy="0 0 0" xyz="0 0 0"/>
+          <geometry>
+            <sphere radius="${foot_radius}"/>
           </geometry>
           <material name="orange"/>
@@ -194,146 +330,15 @@
           <origin rpy="0 0 0" xyz="0 0 0"/>
           <geometry>
-            <sphere radius="0.021"/>
+            <sphere radius="${foot_radius}"/>
           </geometry>
         </collision>
         <xacro:inertial_foot></xacro:inertial_foot>
       </link>
-    <!-- *********** BR_hip ********** -->
-    <link name="BR_hip_link">
-        <visual>
-            <origin xyz="0 0 0" rpy="0 0 0"/>
-            <geometry>
-                <xacro:rightHip_mesh></xacro:rightHip_mesh>
-            </geometry>
-            <material name="red">
-                <color rgba="0.8 0.2 0.2 1"/>
-            </material>
-        </visual>
-        <collision>
-            <origin xyz="0 0 0" rpy="0 0 0"/>
-            <geometry>
-                <xacro:rightHip_mesh></xacro:rightHip_mesh>
-            </geometry>
-        </collision>
-        <xacro:inertial_right_hip></xacro:inertial_right_hip>
-    </link>
-    <!-- *********** BR_uleg ********** -->
-    <link name="BR_uleg_link">
-        <visual>
-            <origin xyz="0 0 0" rpy="0 0 0"/>
-            <geometry>
-                <xacro:rightUleg_mesh></xacro:rightUleg_mesh>
-            </geometry>
-            <material name="orange">
-                <color rgba="0.8 0.5 0.8 1"/>
-            </material>
-        </visual>
-        <collision>
-            <origin xyz="0 0 0" rpy="0 0 0"/>
-            <geometry>
-                <xacro:rightUleg_mesh></xacro:rightUleg_mesh>
-            </geometry>
-        </collision>
-        <xacro:inertial_right_uleg></xacro:inertial_right_uleg>
-    </link>
-    <!-- *********** BR_lleg ********** -->
-    <link name="BR_lleg_link">
-        <visual>
-            <origin xyz="0 0 0" rpy="0 0 0"/>
-            <geometry>
-                <xacro:lleg_mesh></xacro:lleg_mesh>
-            </geometry>
-            <material name="yellow">
-                <color rgba="0.8 1.0 0.1 1"/>
-            </material>
-        </visual>
-        <collision>
-            <origin xyz="0 0 0" rpy="0 0 0"/>
-            <geometry>
-                <xacro:lleg_mesh></xacro:lleg_mesh>
-            </geometry>
-        </collision>
-        <xacro:inertial_right_lleg></xacro:inertial_right_lleg>
-    </link>
-    <!-- *********** BR FOOT ********** -->
-    <link name="BR_foot">
-        <visual>
-          <origin rpy="0 0 0" xyz="0 0 0"/>
-          <geometry>
-            <sphere radius="0.02"/>
-          </geometry>
-          <material name="orange"/>
-        </visual>
-        <collision>
-          <origin rpy="0 0 0" xyz="0 0 0"/>
-          <geometry>
-            <sphere radius="0.021"/>
-          </geometry>
-        </collision>
-        <xacro:inertial_foot></xacro:inertial_foot>
-      </link>
-    <!-- *********** BL_hip ********** -->
-    <link name="BL_hip_link">
-        <visual>
-            <origin xyz="0 0 0" rpy="0 0 0"/>
-            <geometry>
-                <xacro:leftHip_mesh></xacro:leftHip_mesh>
-            </geometry>
-            <material name="red">
-                <color rgba="0.8 0.2 0.2 1"/>
-            </material>
-        </visual>
-        <collision>
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
File: hyperdog_gazebo_sim/description/physics.xacro (robot description, xacro)
@@ -1,21 +1,5 @@
 <?xml version="1.0"?>
 <robot xmlns:xacro="http://www.ros.org/wiki/xacro" >
-    <!-- configure inertia -->
-    <xacro:property name="body_mass" value="4"/>
-    <xacro:property name="body_x_len" value="0.28"/>
-    <xacro:property name="body_y_len" value="0.172"/>
-    <xacro:property name="body_z_len" value="0.04"/>
-    <xacro:property name="hip_mass" value="0.3"/>
-    <xacro:property name="hip_x_len" value="0.05"/>
-    <xacro:property name="hip_y_len" value="0.03"/>
-    <xacro:property name="hip_z_len" value="0.04"/>
-    <xacro:property name="uleg_mass" value="0.5"/>
-    <xacro:property name="uleg_x_len" value="0.1"/>
-    <xacro:property name="uleg_y_len" value="0.02"/>
-    <xacro:property name="uleg_z_len" value="0.02"/>
-    <xacro:property name="lleg_mass" value="0.3"/>
-    <xacro:property name="lleg_x_len" value="0.1"/>
-    <xacro:property name="lleg_y_len" value="0.01"/>
-    <xacro:property name="lleg_z_len" value="0.01"/>
+    <xacro:include filename="consts.xacro" />
     <!--  BODY -->
     <xacro:macro name="inertial_body">
@@ -23,11 +7,7 @@
             <origin xyz="-0.006 0.00633 0.00214" rpy="0 0 0"/> <!-- 0.006, -0.000233, 0.00214 -->
             <mass value="${body_mass}" />
-            <inertia ixx="${(1/12) * body_mass * (body_y_len * body_y_len + body_z_len * body_z_len)}" ixy="0.0" ixz="0.0"
-                     iyy="${(1/12) * body_mass * (body_x_len * body_x_len + body_z_len * body_z_len)}" iyz="0.0"
-                     izz="${(1/12) * body_mass * (body_x_len * body_x_len + body_y_len * body_y_len)}" />
-            <!-- <mass value="2.0"/>
-            <inertia ixx="0.00728" ixy="0.00003" ixz="0.00073"
-                     iyy="0.01641" iyz="0.00013" izz="0.01965"/>
-             -->
+            <inertia ixx="${(1/12) * body_mass * (body_inertia_y_len * body_inertia_y_len + body_inertia_z_len * body_inertia_z_len)}" ixy="0.0" ixz="0.0"
+                     iyy="${(1/12) * body_mass * (body_inertia_x_len * body_inertia_x_len + body_inertia_z_len * body_inertia_z_len)}" iyz="0.0"
+                     izz="${(1/12) * body_mass * (body_inertia_x_len * body_inertia_x_len + body_inertia_y_len * body_inertia_y_len)}" />
         </inertial>
     </xacro:macro>
@@ -37,10 +17,7 @@
             <origin xyz="0.0 -0.02 0.01" rpy="0 0 0"/>
             <mass value="${hip_mass}" />
-            <inertia ixx="${(1/12) * hip_mass * (hip_y_len * hip_y_len + hip_z_len * hip_z_len)}" ixy="0.0" ixz="0.0"
-                     iyy="${(1/12) * hip_mass * (hip_x_len * hip_x_len + hip_z_len * hip_z_len)}" iyz="0.0"
-                     izz="${(1/12) * hip_mass * (hip_x_len * hip_x_len + hip_y_len * hip_y_len)}" />
-            <!-- <mass value="0.25"/>
-            <inertia ixx="0.00199" ixy="0.00339" ixz="0.00075"
-                    iyy="0.0078" iyz="0.00034" izz="0.00943"/> -->
+            <inertia ixx="${(1/12) * hip_mass * (hip_inertia_y_len * hip_inertia_y_len + hip_inertia_z_len * hip_inertia_z_len)}" ixy="0.0" ixz="0.0"
+                     iyy="${(1/12) * hip_mass * (hip_inertia_x_len * hip_inertia_x_len + hip_inertia_z_len * hip_inertia_z_len)}" iyz="0.0"
+                     izz="${(1/12) * hip_mass * (hip_inertia_x_len * hip_inertia_x_len + hip_inertia_y_len * hip_inertia_y_len)}" />
         </inertial>
     </xacro:macro>
@@ -49,10 +26,7 @@
             <origin xyz="0.0 0.02 0.01" rpy="0 0 0"/>
             <mass value="${hip_mass}" />
-            <inertia ixx="${(1/12) * hip_mass * (hip_y_len * hip_y_len + hip_z_len * hip_z_len)}" ixy="0.0" ixz="0.0"
-                     iyy="${(1/12) * hip_mass * (hip_x_len * hip_x_len + hip_z_len * hip_z_len)}" iyz="0.0"
-                     izz="${(1/12) * hip_mass * (hip_x_len * hip_x_len + hip_y_len * hip_y_len)}" />
-            <!-- <mass value="0.25"/>
-            <inertia ixx="0.00199" ixy="0.00339" ixz="0.00075"
-                     iyy="0.0078" iyz="0.00034" izz="0.00943"/> -->
+            <inertia ixx="${(1/12) * hip_mass * (hip_inertia_y_len * hip_inertia_y_len + hip_inertia_z_len * hip_inertia_z_len)}" ixy="0.0" ixz="0.0"
+                     iyy="${(1/12) * hip_mass * (hip_inertia_x_len * hip_inertia_x_len + hip_inertia_z_len * hip_inertia_z_len)}" iyz="0.0"
+                     izz="${(1/12) * hip_mass * (hip_inertia_x_len * hip_inertia_x_len + hip_inertia_y_len * hip_inertia_y_len)}" />
         </inertial>
     </xacro:macro>
@@ -61,11 +35,11 @@
         <inertial>
             <origin xyz="-0.02 0.02 0.0" rpy="0 0 0"/>
-            <!-- <mass value="${uleg_mass}" />
-            <inertia ixx="${(1/12) * uleg_mass * (uleg_y_len * uleg_y_len + uleg_z_len * uleg_z_len)}" ixy="0.0" ixz="0.0"
+            <mass value="${uleg_mass}" />
+            <!-- <inertia ixx="${(1/12) * uleg_mass * (uleg_y_len * uleg_y_len + uleg_z_len * uleg_z_len)}" ixy="0.0" ixz="0.0"
                      iyy="${(1/12) * uleg_mass * (uleg_x_len * uleg_x_len + uleg_z_len * uleg_z_len)}" iyz="0.0"
                      izz="${(1/12) * uleg_mass * (uleg_x_len * uleg_x_len + uleg_y_len * uleg_y_len)}" /> -->
             <mass value="0.35"/>
-            <inertia ixx="0.007467" ixy="0.009383" ixz="0.000515"
-                     iyy="0.012791" iyz="0.000298" izz="0.019903"/>
+            <inertia ixx="0.000418" ixy="-0.000078" ixz="-0.00019"
+                     iyy="0.000484" iyz="0.000051" izz="0.000566"/>
         </inertial>
     </xacro:macro>
@@ -78,6 +52,6 @@
                      izz="${(1/12) * uleg_mass * (uleg_x_len * uleg_x_len + uleg_y_len * uleg_y_len)}" /> -->
             <mass value="0.35"/>
-            <inertia ixx="0.007467" ixy="0.009383" ixz="0.000515"
-                    iyy="0.012791" iyz="0.000298" izz="0.019903"/>
+            <inertia ixx="0.000418" ixy="0.000078" ixz="-0.00019"
+                     iyy="0.000484" iyz="-0.000051" izz="0.000566"/>
         </inertial>
     </xacro:macro>
@@ -85,5 +59,5 @@
     <xacro:macro name="inertial_right_lleg">
         <inertial>
-            <origin xyz="0.05 0.0 -0.0" rpy="0 0 0"/>
+            <origin xyz="0.05 0.0 0.0" rpy="0 0 0"/>
             <!-- <mass value="${lleg_mass}" />
             <inertia ixx="${(1/12) * lleg_mass * (lleg_y_len * lleg_y_len + lleg_z_len * lleg_z_len)}" ixy="0.0" ixz="0.0"
@@ -91,11 +65,11 @@
                      izz="${(1/12) * lleg_mass * (lleg_x_len * lleg_x_len + lleg_y_len * lleg_y_len)}" /> -->
             <mass value="0.24"/>
-            <inertia ixx="0.01273" ixy="0.01054" ixz="0.00877"
-                    iyy="0.02196" iyz="0.00602" izz="0.02318"/>
+            <inertia ixx="0.0.00056" ixy="0.0" ixz="0.00035"
+                    iyy="0.0008" iyz="0.0" izz="0.00026"/>
         </inertial>
     </xacro:macro>
     <xacro:macro name="inertial_left_lleg">
         <inertial>
-            <origin xyz="0.05 0.0 -0.0" rpy="0 0 0"/>
+            <origin xyz="0.05 0.0 0.0" rpy="0 0 0"/>
             <!-- <mass value="${lleg_mass}" />
             <inertia ixx="${(1/12) * lleg_mass * (lleg_y_len * lleg_y_len + lleg_z_len * lleg_z_len)}" ixy="0.0" ixz="0.0"
@@ -103,12 +77,16 @@
                      izz="${(1/12) * lleg_mass * (lleg_x_len * lleg_x_len + lleg_y_len * lleg_y_len)}" /> -->
             <mass value="0.24"/>
-            <inertia ixx="0.01273" ixy="0.01054" ixz="0.00877"
-                    iyy="0.02196" iyz="0.00602" izz="0.02318"/>
+            <inertia ixx="0.0.00056" ixy="0.0" ixz="0.00035"
+                    iyy="0.0008" iyz="0.0" izz="0.00026"/>
         </inertial>
     </xacro:macro>
+    <!-- FOOT -->
     <xacro:macro name="inertial_foot">
         <inertial>
-            <mass value="0.06"/>
-            <inertia ixx="9.6e-06" ixy="0.0" ixz="0.0" iyy="9.6e-06" iyz="0.0" izz="9.6e-06"/>
+            <origin xyz="0.0 0.0 0.0" rpy="0 0 0"/>
+            <mass value="${foot_mass}"/>
+            <inertia ixx="${2.0/5.0 * foot_radius * foot_radius * foot_mass}" ixy="0.0" ixz="0.0"
+                     iyy="${2.0/5.0 * foot_radius * foot_radius * foot_mass}" iyz="0.0"
+                     izz="${2.0/5.0 * foot_radius * foot_radius * foot_mass}"/>
         </inertial>
     </xacro:macro>
