Commit message: deleted hyperdog_gazebo_joint_cmd pkg, added gazebo joint cmd node to hyperdog_gazebo_sim pkg in cpp

File: hyperdog_gazebo_sim/description/consts.xacro (robot description, xacro)
@@ -13,11 +13,11 @@
     <xacro:property name="use_dynamics" value="true"/>
     <xacro:macro name="hip_joint_dynamics">
-        <dynamics damping="1" friction="10"/>
+        <dynamics damping="10" friction="1000"/>
     </xacro:macro>
     <xacro:macro name="uleg_joint_dynamics">
-        <dynamics damping="1" friction="10"/>
+        <dynamics damping="10" friction="1000"/>
     </xacro:macro>
     <xacro:macro name="lleg_joint_dynamics">
-        <dynamics damping="1" friction="10"/>
+        <dynamics damping="10" friction="10000"/>
     </xacro:macro>
     <!-- configure inertia -->
@@ -34,8 +34,8 @@
     <xacro:property name="uleg_inertia_y_len" value="0.01"/>
     <xacro:property name="uleg_inertia_z_len" value="0.01"/>
-    <xacro:property name="lleg_mass" value="0.3"/>
-    <xacro:property name="lleg_inertia_x_len" value="0.1"/>
-    <xacro:property name="lleg_inertia_y_len" value="0.01"/>
-    <xacro:property name="lleg_inertia_z_len" value="0.01"/>
+    <xacro:property name="lleg_mass" value="0.2"/>
+    <xacro:property name="lleg_inertia_x_len" value="0.08"/>
+    <xacro:property name="lleg_inertia_y_len" value="0.001"/>
+    <xacro:property name="lleg_inertia_z_len" value="0.005"/>
     <!-- feet -->
     <xacro:property name="foot_mass" value="0.1"/>

File: hyperdog_gazebo_sim/description/hyperdog_gazebo.xacro (robot description, xacro)
@@ -14,6 +14,6 @@
         <mu1>0.2</mu1>
         <mu2>0.2</mu2>
-        <!-- <kp value="1000000.0"/>
-        <kd value="1.0"/> -->
+        <kp value="1000000.0"/>
+        <kd value="1.0"/>
         <!-- <maxVel>0.0</maxVel> -->
         <material>Gazebo/PioneerBody</material>
@@ -22,6 +22,6 @@
         <mu1>0.2</mu1>
         <mu2>0.2</mu2>
-        <!-- <kp value="2147483647.0"/>
-        <kd value="1.0"/> -->
+        <kp value="2147483647.0"/>
+        <kd value="1.0"/>
         <!-- <maxVel>0.0</maxVel> -->
         <!-- <self_collide>1</self_collide> -->
@@ -33,6 +33,6 @@
         <mu1>0.2</mu1>
         <mu2>0.2</mu2>
-        <!-- <kp>1000000.0</kp>
-        <kd>1.0</kd> -->
+        <kp>1000000.0</kp>
+        <kd>1.0</kd>
         <!-- <maxVel>0.0</maxVel> -->
         <!-- <self_collide>1</self_collide>  -->
@@ -42,10 +42,10 @@
     </xacro:macro>
     <xacro:macro name="gz_foot">
-        <mu1>1.0</mu1>
-        <mu2>1.0</mu2>
+        <mu1>0.9</mu1>
+        <mu2>0.9</mu2>
         <kp value="1000000.0" />
         <kd value="100.0" />
-        <!-- <maxVel>0.0</maxVel> -->
-        <!-- <self_collide>1</self_collide> -->
+        <maxVel>0.0</maxVel>
+        <self_collide>1</self_collide>
         <minDepth>0.001</minDepth>
         <material>Gazebo/DarkGrey</material>

File: hyperdog_gazebo_sim/description/physics.xacro (robot description, xacro)
@@ -48,7 +48,7 @@
             <origin xyz="-0.02 -0.02 0.0" rpy="0 0 0"/>
             <!-- <mass value="${uleg_mass}"/>
-            <inertia ixx="${(1/12) * uleg_mass * (uleg_y_len * uleg_y_len + uleg_z_len * uleg_z_len)}" ixy="0.0" ixz="0.0"
-                     iyy="${(1/12) * uleg_mass * (uleg_x_len * uleg_x_len + uleg_z_len * uleg_z_len)}" iyz="0.0"
-                     izz="${(1/12) * uleg_mass * (uleg_x_len * uleg_x_len + uleg_y_len * uleg_y_len)}" /> -->
+            <inertia ixx="${(1/12) * uleg_mass * (uleg_inertia_y_len * uleg_inertia_y_len + uleg_inertia_z_len * uleg_inertia_z_len)}" ixy="0.0" ixz="0.0"
+                     iyy="${(1/12) * uleg_mass * (uleg_inertia_x_len * uleg_inertia_x_len + uleg_inertia_z_len * uleg_inertia_z_len)}" iyz="0.0"
+                     izz="${(1/12) * uleg_mass * (uleg_inertia_x_len * uleg_inertia_x_len + uleg_inertia_y_len * uleg_inertia_y_len)}" /> -->
             <mass value="0.35"/>
             <inertia ixx="0.000418" ixy="0.000078" ixz="-0.00019"
@@ -60,11 +60,11 @@
         <inertial>
             <origin xyz="0.05 0.0 0.0" rpy="0 0 0"/>
-            <!-- <mass value="${lleg_mass}" />
-            <inertia ixx="${(1/12) * lleg_mass * (lleg_y_len * lleg_y_len + lleg_z_len * lleg_z_len)}" ixy="0.0" ixz="0.0"
-                     iyy="${(1/12) * lleg_mass * (lleg_x_len * lleg_x_len + lleg_z_len * lleg_z_len)}" iyz="0.0"
-                     izz="${(1/12) * lleg_mass * (lleg_x_len * lleg_x_len + lleg_y_len * lleg_y_len)}" /> -->
-            <mass value="0.24"/>
+            <mass value="${lleg_mass}" />
+            <inertia ixx="${(1/12) * lleg_mass * (lleg_inertia_y_len * lleg_inertia_y_len + lleg_inertia_z_len * lleg_inertia_z_len)}" ixy="0.0" ixz="0.0"
+                     iyy="${(1/12) * lleg_mass * (lleg_inertia_x_len * lleg_inertia_x_len + lleg_inertia_z_len * lleg_inertia_z_len)}" iyz="0.0"
+                     izz="${(1/12) * lleg_mass * (lleg_inertia_x_len * lleg_inertia_x_len + lleg_inertia_y_len * lleg_inertia_y_len)}" />
+            <!-- <mass value="0.24"/>
             <inertia ixx="0.0.00056" ixy="0.0" ixz="0.00035"
-                    iyy="0.0008" iyz="0.0" izz="0.00026"/>
+                    iyy="0.0008" iyz="0.0" izz="0.00026"/> -->
         </inertial>
     </xacro:macro>
@@ -72,11 +72,11 @@
         <inertial>
             <origin xyz="0.05 0.0 0.0" rpy="0 0 0"/>
-            <!-- <mass value="${lleg_mass}" />
-            <inertia ixx="${(1/12) * lleg_mass * (lleg_y_len * lleg_y_len + lleg_z_len * lleg_z_len)}" ixy="0.0" ixz="0.0"
-                     iyy="${(1/12) * lleg_mass * (lleg_x_len * lleg_x_len + lleg_z_len * lleg_z_len)}" iyz="0.0"
-                     izz="${(1/12) * lleg_mass * (lleg_x_len * lleg_x_len + lleg_y_len * lleg_y_len)}" /> -->
-            <mass value="0.24"/>
+            <mass value="${lleg_mass}" />
+            <inertia ixx="${(1/12) * lleg_mass * (lleg_inertia_y_len * lleg_inertia_y_len + lleg_inertia_z_len * lleg_inertia_z_len)}" ixy="0.0" ixz="0.0"
+                     iyy="${(1/12) * lleg_mass * (lleg_inertia_x_len * lleg_inertia_x_len + lleg_inertia_z_len * lleg_inertia_z_len)}" iyz="0.0"
+                     izz="${(1/12) * lleg_mass * (lleg_inertia_x_len * lleg_inertia_x_len + lleg_inertia_y_len * lleg_inertia_y_len)}" />
+            <!-- <mass value="0.24"/>
             <inertia ixx="0.0.00056" ixy="0.0" ixz="0.00035"
-                    iyy="0.0008" iyz="0.0" izz="0.00026"/>
+                    iyy="0.0008" iyz="0.0" izz="0.00026"/> -->
         </inertial>
     </xacro:macro>
@@ -86,7 +86,10 @@
             <origin xyz="0.0 0.0 0.0" rpy="0 0 0"/>
             <mass value="${foot_mass}"/>
-            <inertia ixx="${2.0/5.0 * foot_radius * foot_radius * foot_mass}" ixy="0.0" ixz="0.0"
-                     iyy="${2.0/5.0 * foot_radius * foot_radius * foot_mass}" iyz="0.0"
-                     izz="${2.0/5.0 * foot_radius * foot_radius * foot_mass}"/>
+            <!-- <inertia ixx="${2/5 * foot_radius * foot_radius * foot_mass}" ixy="0.0" ixz="0.0"
+                     iyy="${2/5 * foot_radius * foot_radius * foot_mass}" iyz="0.0"
+                     izz="${2/5 * foot_radius * foot_radius * foot_mass}"/> -->
+            <inertia ixx="${(1/12) * foot_mass * (0.01 * 0.01 + 0.01 * 0.01)}" ixy="0.0" ixz="0.0"
+                    iyy="${(1/12) * foot_mass * (0.01 * 0.01 + 0.01 * 0.01)}" iyz="0.0"
+                    izz="${(1/12) * foot_mass * (0.01 * 0.01 + 0.01 * 0.01)}" />
         </inertial>
     </xacro:macro>

Commit message: updated inertias of links

File: hyperdog_gazebo_sim/description/consts.xacro (robot description, xacro)
@@ -13,14 +13,14 @@
     <xacro:property name="use_dynamics" value="true"/>
     <xacro:macro name="hip_joint_dynamics">
-        <dynamics damping="10" friction="1000"/>
+        <dynamics damping="0.01" friction="10000"/>
     </xacro:macro>
     <xacro:macro name="uleg_joint_dynamics">
-        <dynamics damping="10" friction="1000"/>
+        <dynamics damping="0.01" friction="10000"/>
     </xacro:macro>
     <xacro:macro name="lleg_joint_dynamics">
-        <dynamics damping="10" friction="10000"/>
+        <dynamics damping="0.01" friction="10000"/>
     </xacro:macro>
     <!-- configure inertia -->
-    <xacro:property name="body_mass" value="15"/>
+    <xacro:property name="body_mass" value="3"/>
     <xacro:property name="body_inertia_x_len" value="0.28"/>
     <xacro:property name="body_inertia_y_len" value="0.172"/>

File: hyperdog_gazebo_sim/description/hyperdog_gazebo.xacro (robot description, xacro)
@@ -14,7 +14,8 @@
         <mu1>0.2</mu1>
         <mu2>0.2</mu2>
-        <kp value="1000000.0"/>
+        <kp value="2147483647.0"/>
         <kd value="1.0"/>
-        <!-- <maxVel>0.0</maxVel> -->
+        <maxVel>0.01</maxVel>
+        <self_collide>1</self_collide>
         <material>Gazebo/PioneerBody</material>
     </xacro:macro>
@@ -24,6 +25,6 @@
         <kp value="2147483647.0"/>
         <kd value="1.0"/>
-        <!-- <maxVel>0.0</maxVel> -->
-        <!-- <self_collide>1</self_collide> -->
+        <maxVel>0.01</maxVel>
+        <self_collide>1</self_collide>
         <material>Gazebo/Orange</material>
         <!-- <implicitSpringDamper>1</implicitSpringDamper>
@@ -33,9 +34,11 @@
         <mu1>0.2</mu1>
         <mu2>0.2</mu2>
-        <kp>1000000.0</kp>
+        <fdir1>1 0 0</fdir1>
+        <kp>2147483647.0</kp>
         <kd>1.0</kd>
-        <!-- <maxVel>0.0</maxVel> -->
-        <!-- <self_collide>1</self_collide>  -->
+        <maxVel>0.01</maxVel>
+        <self_collide>1</self_collide>
         <material>Gazebo/DarkYellow</material>
+        <minDepth>0.001</minDepth>
         <!-- <implicitSpringDamper>1</implicitSpringDamper>
         <springStiffness>100</springStiffness> -->
@@ -44,9 +47,12 @@
         <mu1>0.9</mu1>
         <mu2>0.9</mu2>
-        <kp value="1000000.0" />
+        <fdir1>1 1 0</fdir1>
+        <kp value="2147483647.0" />
         <kd value="100.0" />
-        <maxVel>0.0</maxVel>
+        <maxVel>0.01</maxVel>
         <self_collide>1</self_collide>
         <minDepth>0.001</minDepth>
+        <restitution_coefficient>1</restitution_coefficient>
+        <threshold>0</threshold>
         <material>Gazebo/DarkGrey</material>
     </xacro:macro>
@@ -57,4 +63,5 @@
         <!-- <kp>1000000.0</kp>
         <kd>1.0</kd> -->
+        <maxVel>0.01</maxVel>
         <material>Gazebo/DarkGrey  </material>
     </gazebo>

File: hyperdog_gazebo_sim/description/hyperdog_urdf_links.xacro (robot description, xacro)
@@ -298,4 +298,13 @@
             <sphere radius="${foot_radius}"/>
           </geometry>
+          <surface>
+            <friction>
+                <ode>
+                    <mu>1</mu>
+                    <mu2>1</mu2>
+                    <fdir1>1 0 0</fdir1>
+                </ode>
+            </friction>
+        </surface>
         </collision>
         <xacro:inertial_foot></xacro:inertial_foot>
@@ -315,4 +324,13 @@
             <sphere radius="${foot_radius}"/>
           </geometry>
+          <surface>
+            <friction>
+                <ode>
+                    <mu>1</mu>
+                    <mu2>1</mu2>
+                    <fdir1>1 0 0</fdir1>
+                </ode>
+            </friction>
+        </surface>
         </collision>
         <xacro:inertial_foot></xacro:inertial_foot>
@@ -332,4 +350,13 @@
             <sphere radius="${foot_radius}"/>
           </geometry>
+          <surface>
+            <friction>
+                <ode>
+                    <mu>1</mu>
+                    <mu2>1</mu2>
+                    <fdir1>1 0 0</fdir1>
+                </ode>
+            </friction>
+        </surface>
         </collision>
         <xacro:inertial_foot></xacro:inertial_foot>
@@ -349,4 +376,13 @@
             <sphere radius="${foot_radius}"/>
           </geometry>
+          <surface>
+            <friction>
+                <ode>
+                    <mu>1</mu>
+                    <mu2>1</mu2>
+                    <fdir1>1 0 0</fdir1>
+                </ode>
+            </friction>
+        </surface>
         </collision>
         <xacro:inertial_foot></xacro:inertial_foot>

File: hyperdog_gazebo_sim/description/physics.xacro (robot description, xacro)
@@ -7,7 +7,5 @@
             <origin xyz="-0.006 0.00633 0.00214" rpy="0 0 0"/> <!-- 0.006, -0.000233, 0.00214 -->
             <mass value="${body_mass}" />
-            <inertia ixx="${(1/12) * body_mass * (body_inertia_y_len * body_inertia_y_len + body_inertia_z_len * body_inertia_z_len)}" ixy="0.0" ixz="0.0"
-                     iyy="${(1/12) * body_mass * (body_inertia_x_len * body_inertia_x_len + body_inertia_z_len * body_inertia_z_len)}" iyz="0.0"
-                     izz="${(1/12) * body_mass * (body_inertia_x_len * body_inertia_x_len + body_inertia_y_len * body_inertia_y_len)}" />
+            <inertia  ixx="0.011396658109874464" ixy="0" ixz="0" iyy="0.05486450023370329" iyz="0" izz="0.06098759357764758" />
         </inertial>
     </xacro:macro>
@@ -17,7 +15,5 @@
             <origin xyz="0.0 -0.02 0.01" rpy="0 0 0"/>
             <mass value="${hip_mass}" />
-            <inertia ixx="${(1/12) * hip_mass * (hip_inertia_y_len * hip_inertia_y_len + hip_inertia_z_len * hip_inertia_z_len)}" ixy="0.0" ixz="0.0"
-                     iyy="${(1/12) * hip_mass * (hip_inertia_x_len * hip_inertia_x_len + hip_inertia_z_len * hip_inertia_z_len)}" iyz="0.0"
-                     izz="${(1/12) * hip_mass * (hip_inertia_x_len * hip_inertia_x_len + hip_inertia_y_len * hip_inertia_y_len)}" />
+            <inertia  ixx="0.000785664594069212" ixy="0" ixz="0" iyy="0.00028126771524959764" iyz="0" izz="0.0007138119943369485" />
         </inertial>
     </xacro:macro>
@@ -26,7 +22,5 @@
             <origin xyz="0.0 0.02 0.01" rpy="0 0 0"/>
             <mass value="${hip_mass}" />
-            <inertia ixx="${(1/12) * hip_mass * (hip_inertia_y_len * hip_inertia_y_len + hip_inertia_z_len * hip_inertia_z_len)}" ixy="0.0" ixz="0.0"
-                     iyy="${(1/12) * hip_mass * (hip_inertia_x_len * hip_inertia_x_len + hip_inertia_z_len * hip_inertia_z_len)}" iyz="0.0"
-                     izz="${(1/12) * hip_mass * (hip_inertia_x_len * hip_inertia_x_len + hip_inertia_y_len * hip_inertia_y_len)}" />
+            <inertia  ixx="0.000785664594069212" ixy="0" ixz="0" iyy="0.00028126771524959764" iyz="0" izz="0.0007138119943369485" />
         </inertial>
     </xacro:macro>
@@ -36,10 +30,5 @@
             <origin xyz="-0.02 0.02 0.0" rpy="0 0 0"/>
             <mass value="${uleg_mass}" />
-            <!-- <inertia ixx="${(1/12) * uleg_mass * (uleg_y_len * uleg_y_len + uleg_z_len * uleg_z_len)}" ixy="0.0" ixz="0.0"
-                     iyy="${(1/12) * uleg_mass * (uleg_x_len * uleg_x_len + uleg_z_len * uleg_z_len)}" iyz="0.0"
-                     izz="${(1/12) * uleg_mass * (uleg_x_len * uleg_x_len + uleg_y_len * uleg_y_len)}" /> -->
-            <mass value="0.35"/>
-            <inertia ixx="0.000418" ixy="-0.000078" ixz="-0.00019"
-                     iyy="0.000484" iyz="0.000051" izz="0.000566"/>
+            <inertia  ixx="0.0005320036781441746" ixy="0" ixz="0" iyy="0.00178632152356757" iyz="0" izz="0.002124721126775121" />
         </inertial>
     </xacro:macro>
@@ -47,11 +36,6 @@
         <inertial>
             <origin xyz="-0.02 -0.02 0.0" rpy="0 0 0"/>
-            <!-- <mass value="${uleg_mass}"/>
-            <inertia ixx="${(1/12) * uleg_mass * (uleg_inertia_y_len * uleg_inertia_y_len + uleg_inertia_z_len * uleg_inertia_z_len)}" ixy="0.0" ixz="0.0"
-                     iyy="${(1/12) * uleg_mass * (uleg_inertia_x_len * uleg_inertia_x_len + uleg_inertia_z_len * uleg_inertia_z_len)}" iyz="0.0"
-                     izz="${(1/12) * uleg_mass * (uleg_inertia_x_len * uleg_inertia_x_len + uleg_inertia_y_len * uleg_inertia_y_len)}" /> -->
-            <mass value="0.35"/>
-            <inertia ixx="0.000418" ixy="0.000078" ixz="-0.00019"
-                     iyy="0.000484" iyz="-0.000051" izz="0.000566"/>
+            <mass value="${uleg_mass}"/>
+            <inertia  ixx="0.0005320036934665719" ixy="0" ixz="0" iyy="0.0017863215388899672" iyz="0" izz="0.002124721126775121" />
         </inertial>
     </xacro:macro>
@@ -61,10 +45,5 @@
             <origin xyz="0.05 0.0 0.0" rpy="0 0 0"/>
             <mass value="${lleg_mass}" />
-            <inertia ixx="${(1/12) * lleg_mass * (lleg_inertia_y_len * lleg_inertia_y_len + lleg_inertia_z_len * lleg_inertia_z_len)}" ixy="0.0" ixz="0.0"
-                     iyy="${(1/12) * lleg_mass * (lleg_inertia_x_len * lleg_inertia_x_len + lleg_inertia_z_len * lleg_inertia_z_len)}" iyz="0.0"
-                     izz="${(1/12) * lleg_mass * (lleg_inertia_x_len * lleg_inertia_x_len + lleg_inertia_y_len * lleg_inertia_y_len)}" />
-            <!-- <mass value="0.24"/>
-            <inertia ixx="0.0.00056" ixy="0.0" ixz="0.00035"
-                    iyy="0.0008" iyz="0.0" izz="0.00026"/> -->
+            <inertia  ixx="6.323427512607013e-05" ixy="0" ixz="0" iyy="0.0006549703843792289" iyz="0" izz="0.0006232548592531587" />
         </inertial>
     </xacro:macro>
@@ -73,10 +52,5 @@
             <origin xyz="0.05 0.0 0.0" rpy="0 0 0"/>
             <mass value="${lleg_mass}" />
-            <inertia ixx="${(1/12) * lleg_mass * (lleg_inertia_y_len * lleg_inertia_y_len + lleg_inertia_z_len * lleg_inertia_z_len)}" ixy="0.0" ixz="0.0"
-                     iyy="${(1/12) * lleg_mass * (lleg_inertia_x_len * lleg_inertia_x_len + lleg_inertia_z_len * lleg_inertia_z_len)}" iyz="0.0"
-                     izz="${(1/12) * lleg_mass * (lleg_inertia_x_len * lleg_inertia_x_len + lleg_inertia_y_len * lleg_inertia_y_len)}" />
-            <!-- <mass value="0.24"/>
-            <inertia ixx="0.0.00056" ixy="0.0" ixz="0.00035"
-                    iyy="0.0008" iyz="0.0" izz="0.00026"/> -->
+            <inertia  ixx="6.323427512607013e-05" ixy="0" ixz="0" iyy="0.0006549703843792289" iyz="0" izz="0.0006232548592531587" />
         </inertial>
     </xacro:macro>
@@ -86,7 +60,4 @@
             <origin xyz="0.0 0.0 0.0" rpy="0 0 0"/>
             <mass value="${foot_mass}"/>
-            <!-- <inertia ixx="${2/5 * foot_radius * foot_radius * foot_mass}" ixy="0.0" ixz="0.0"
-                     iyy="${2/5 * foot_radius * foot_radius * foot_mass}" iyz="0.0"
-                     izz="${2/5 * foot_radius * foot_radius * foot_mass}"/> -->
             <inertia ixx="${(1/12) * foot_mass * (0.01 * 0.01 + 0.01 * 0.01)}" ixy="0.0" ixz="0.0"
                     iyy="${(1/12) * foot_mass * (0.01 * 0.01 + 0.01 * 0.01)}" iyz="0.0"
