Commit message: Add self-righting, robustness campaign, new worlds, RViz markers and bring-up tools
Self-righting (hyperdog_locomotion):
- New SELF_RIGHT mode: after a fall the robot waits in damping until it is at
  rest, then rolls itself onto its belly with the lower side legs, stands up and
  resumes the commanded mode. On its back, a fast kick tips it onto a side first.
  Gives up after max_attempts (damping). All parameters in self_righting.*.
- Validated by the new `fall` scenario (knocked over by a roll torque, dropped on
  its side). Recovery from lying exactly on the back is a documented limitation
  (+-1 rad hip range); `fall_back` scenario reproduces it.

Simulation and validation (hyperdog_gazebo, hyperdog_description):
- Worlds: rough (1-3 cm slabs), stairs (4 cm steps), slippery (mu 0.3 patch).
- Scenarios: speed, robust, fall, fall_back, rough, stairs, slippery. Steps can
  apply roll torques, place the robot via the bridged set_pose service and allow
  a fall (pass when standing upright again at the end).
- robustness_campaign: runs a scenario with randomized payload, foot friction,
  IMU noise, motor current / Kt / friction and command latency; 10/10 pass.
- xacro / launch args for these model variations; BldcImpedanceController gains
  a command_latency parameter.

Tools and visualisation:
- hyperdog/markers MarkerArray (feet, contacts, targets, support polygon, GRFs).
- mit_can_probe (scan / read / zero / low-gain hold) and joint_test (sine
  tracking or torque step with current, saturation and temperature summary).
- docs/hardware_bringup.md: staged bring-up checklist.

Parameters: numeric parameters accept integers (kp: 80) instead of aborting.
Docs: README, architecture, package READMEs and validation reports updated.

Co-Authored-By: Claude Opus 5.5 <noreply@anthropic.com>
Claude-Session: https://claude.ai/code/session_0145DngQugTZatPGg919Q9vX

File: hyperdog_description/urdf/common.xacro (robot description, xacro)
@@ -21,6 +21,5 @@
   <xacro:property name="lleg_mass" value="0.2"/>
   <xacro:property name="foot_mass" value="0.1"/>
-  <!-- foot contact -->
-  <xacro:property name="foot_mu" value="1.0"/>
+  <!-- foot friction (foot_mu) and IMU noise scale (imu_noise_scale) are xacro args of the top level file -->
   <!-- ===== BLDC actuator limits derived from the motor parameter file ===== -->
   <xacro:property name="bldc" value="${xacro.load_yaml(motors_file)['bldc_controller']['ros__parameters']}"/>

File: hyperdog_description/urdf/hyperdog.urdf.xacro (robot description, xacro)
@@ -18,5 +18,15 @@
   <xacro:arg name="controllers_file" default="$(find hyperdog_description)/config/controllers.yaml"/>
   <xacro:arg name="can_interface" default="can0"/>
+  <!-- model variations (robustness testing / payloads) -->
+  <xacro:arg name="payload_mass" default="0.0"/>
+  <xacro:arg name="payload_x" default="0.0"/>
+  <xacro:arg name="payload_y" default="0.0"/>
+  <xacro:arg name="foot_mu" default="1.0"/>
+  <xacro:arg name="imu_noise_scale" default="1.0"/>
+  <!-- optional extra ros2_control parameter file (overrides, e.g. motor variations) -->
+  <xacro:arg name="extra_controller_params" default=""/>
   <xacro:property name="motors_file" value="$(arg motors_file)"/>
+  <xacro:property name="foot_mu" value="$(arg foot_mu)"/>
+  <xacro:property name="imu_noise_scale" value="$(arg imu_noise_scale)"/>
   <xacro:include filename="$(find hyperdog_description)/urdf/common.xacro"/>
   <xacro:include filename="$(find hyperdog_description)/urdf/leg.xacro"/>
@@ -45,4 +55,18 @@
     </inertial>
   </link>
+  <!-- optional payload (point mass) -->
+  <xacro:if value="${$(arg payload_mass) > 0.0}">
+    <joint name="payload_joint" type="fixed">
+      <parent link="base_link"/>
+      <child link="payload_link"/>
+      <origin xyz="$(arg payload_x) $(arg payload_y) 0.08" rpy="0 0 0"/>
+    </joint>
+    <link name="payload_link">
+      <inertial>
+        <mass value="$(arg payload_mass)"/>
+        <inertia ixx="0.001" ixy="0" ixz="0" iyy="0.001" iyz="0" izz="0.001"/>
+      </inertial>
+    </link>
+  </xacro:if>
   <!-- ============================== legs ============================== -->
   <xacro:hyperdog_leg prefix="FR" front="1" left="-1"/>
@@ -66,4 +90,5 @@
   <xacro:hyperdog_ros2_control sim="$(arg sim)" can_interface="$(arg can_interface)"
                                controllers_file="$(arg controllers_file)"
-                               motors_file="$(arg motors_file)"/>
+                               motors_file="$(arg motors_file)"
+                               extra_params="$(arg extra_controller_params)"/>
 </robot>

File: hyperdog_description/urdf/ros2_control.xacro (robot description, xacro)
@@ -5,5 +5,5 @@
   <xacro:property name="init_uleg" value="0.50"/>
   <xacro:property name="init_lleg" value="0.85"/>
-  <xacro:macro name="hyperdog_ros2_control" params="sim can_interface controllers_file motors_file">
+  <xacro:macro name="hyperdog_ros2_control" params="sim can_interface controllers_file motors_file extra_params:=''">
     <ros2_control name="HyperDogSystem" type="system">
       <hardware>
@@ -42,4 +42,7 @@
           <parameters>${controllers_file}</parameters>
           <parameters>${motors_file}</parameters>
+          <xacro:if value="${extra_params != ''}">
+            <parameters>${extra_params}</parameters>
+          </xacro:if>
         </plugin>
       </gazebo>

File: hyperdog_description/urdf/sensors.xacro (robot description, xacro)
@@ -25,12 +25,12 @@
         <imu>
           <angular_velocity>
-            <x><noise type="gaussian"><mean>0</mean><stddev>0.002</stddev></noise></x>
-            <y><noise type="gaussian"><mean>0</mean><stddev>0.002</stddev></noise></y>
-            <z><noise type="gaussian"><mean>0</mean><stddev>0.002</stddev></noise></z>
+            <x><noise type="gaussian"><mean>0</mean><stddev>${0.002 * imu_noise_scale}</stddev></noise></x>
+            <y><noise type="gaussian"><mean>0</mean><stddev>${0.002 * imu_noise_scale}</stddev></noise></y>
+            <z><noise type="gaussian"><mean>0</mean><stddev>${0.002 * imu_noise_scale}</stddev></noise></z>
           </angular_velocity>
           <linear_acceleration>
-            <x><noise type="gaussian"><mean>0</mean><stddev>0.02</stddev></noise></x>
-            <y><noise type="gaussian"><mean>0</mean><stddev>0.02</stddev></noise></y>
-            <z><noise type="gaussian"><mean>0</mean><stddev>0.02</stddev></noise></z>
+            <x><noise type="gaussian"><mean>0</mean><stddev>${0.02 * imu_noise_scale}</stddev></noise></x>
+            <y><noise type="gaussian"><mean>0</mean><stddev>${0.02 * imu_noise_scale}</stddev></noise></y>
+            <z><noise type="gaussian"><mean>0</mean><stddev>${0.02 * imu_noise_scale}</stddev></noise></z>
           </linear_acceleration>
         </imu>
